File: Interconnect.kicad_pcb (KiCad board)
At the start: 2 copper layers, 396.5 x 196.6 mm, 1115 parts, among them J1 9001-11961C00A, J10 SPARE, J11 2x5 2.56mm RA, J12 RJ45, J13 USB-B1HSB6, J14 PJ-082BH, J15 DB9_Female_RA, J16 10x2.54mm, J17 691322310004, J18 10x2.54mm, J19 10x2.54mm, J2 9001-11961C00A, J20 10x2.54mm, J21 10x2.54mm, J22 10x2.54mm, J23 6x2.54mm, J24 6x2.54mm, J25 6x2.54mm, J26 6x2.54mm, J27 6x2.54mm, J28 6x2.54mm, J29 6x2.54mm, J3 7760, J30 6x2.54mm, J31 6x2.54mm, J32 6x2.54mm, J33 Conn_01x04_Female, J4 7760, J5 4 Pins 5.08mm, J6 OSCILLOSCOPE, J7 OSCILLOSCOPE, J8 6 pins 3.81mm, J9 AWG, K1 TQ2-5, K10 TQ2-5, K11 TQ2-5, K12 TQ2-5, K13 TQ2-5, K14 TQ2-5, K15 TQ2-5, K16 TQ2-5, K17 TQ2-5, K18 TQ2-5, K19 TQ2-5, K2 TQ2-5, K20 TQ2-5, K21 TQ2-5, K22 TQ2-5, K23 TQ2-5, K24 TQ2-5, K25 TQ2-5, K26 TQ2-5, K27 TQ2-5, K28 TQ2-5, K29 TQ2-5, K3 G5LE-1, K30 TQ2-5, K31 TQ2-5, K32 TQ2-5, K33 TQ2-5, K34 TQ2-5, K35 TQ2-5, K36 TQ2-5, K37 TQ2-5, K38 TQ2-5, K39 TQ2-5, K4 CPC1706Y, K40 TQ2-5, K41 TQ2-5, K5 TQ2-5, K6 TQ2-5, K7 TQ2-5, K8 TQ2-5, K9 TQ2-5, Q1 2N2222, Q10 2N2222, Q11 2N2222, Q12 2N2222, Q13 2N2222, Q14 2N2222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

Commit message: First try to fit electronic on PCB
Parts:
- removed the D1 at (219.8, 104.8)
- removed the D2 at (243.8, 78.7)
- removed D24: 1N4148, Diode_THT:D_DO-35_SOD27_P7.62mm_Horizontal
- removed the D25 at (99.9, 75.3)
- removed D27, D28, D59, D60, D61, D62, D67, D69, D70, D71, D72, D77, D78, D79, D80, D85: LED, LED_THT:LED_D3.0mm_Clear
- removed the D29 at (59.8, 126.7)
- removed the D3 at (248.9, 72.9)
- removed the D30 at (96.3, 91.6)
- removed the D34 at (53.1, 122.2)
- removed the D35 at (106.5, 79.9)
- removed the D37 at (824.4, 239.4)
- removed the D38 at (824.4, 243.0)
- removed the D39 at (795.6, 271.7)
- removed the D4 at (238.6, 84.6)
- removed the D40 at (784.8, 271.7)
- removed the D41 at (853.0, 224.9)
- removed the D42 at (859.5, 215.4)
- removed the D45 at (865.9, 213.8)
- removed the D46 at (872.4, 208.0)
- removed the D51 at (662.3, 326.9)
- removed the D52 at (656.4, 326.9)
- removed the D53 at (639.5, 347.6)
- removed the D54 at (656.4, 332.4)
- removed the D9 at (202.1, 119.7)
- removed F2: MC000827, SnapEDA Library:MC000827
- removed the NT412 at (200.0, 154.9)
- removed the NT413 at (567.6, -7.06)
- removed the NT414 at (584.0, -12.8)
- removed the NT415 at (590.1, -30.1)
- removed the NT416 at (578.5, -12.8)
- removed the NT417 at (567.6, -4.21)
- removed the NT418 at (200.0, 160.6)
- removed the NT419 at (590.1, -27.3)
- removed the NT420 at (573.1, -9.91)
- removed the NT421 at (590.1, -21.6)
- removed the R1 at (179.6, 122.6)
- removed R105, R106, R107, R108, R113, R115, R116, R117, R118, R123, R124, R125, R126, R131, R30, R37: 220, Resistor_THT:R_Axial_DIN0309_L9.0mm_D3.2mm_P12.70mm_Horizontal
- removed the R11 at (203.0, 99.5)
- removed the R12 at (447.4, 353.6)
- removed R127, R130: 10K, Resistor_THT:R_Axial_DIN0309_L9.0mm_D3.2mm_P12.70mm_Horizontal
- removed the R19 at (472.1, 140.5)
- removed the R26 at (104.5, 110.2)
- removed the R27 at (84.1, 80.7)
- removed the R28 at (37.3, 124.8)
- removed the R35 at (44.8, 118.0)
- removed the R36 at (56.5, 101.7)
- removed the R38 at (44.8, 108.5)
- removed the R4 at (255.8, 191.4)
- removed the R43 at (68.2, 85.4)
- removed the R47 at (837.1, 218.7)
- removed the R48 at (837.1, 223.5)
- removed the R51 at (809.9, 187.3)
- removed the R53 at (859.2, 190.0)
- removed the R55 at (837.1, 228.2)
- removed the R6 at (187.2, 111.0)
- removed the R7 at (255.8, 186.6)
- removed the R9 at (226.4, 73.7)
- removed the R98 at (606.2, 344.7)
- removed the R99 at (668.9, 291.0)
- removed TP181, TP184, TP187, TP188, TP189, TP255, TP256, TP257, TP258, TP259, TP260: TestPoint_Small, Connector_PinHeader_2.54mm:PinHeader_1x01_P2.54mm_Vertical
- removed the TP24 at (589.8, -7.41)
- removed the TP26 at (606.8, -24.8)
- added NT436: M3_4, NetTie:NetTie-2_THT_Pad1.0mm, F.Cu at (-106.7, -62.9)
- added NT437: M3_H4, NetTie:NetTie-2_THT_Pad1.0mm, F.Cu at (-82.5, -63.5)
- added NT438: M2_1, NetTie:NetTie-2_THT_Pad1.0mm, F.Cu at (-105.4, -102.9)
- added NT439: M2_H1, NetTie:NetTie-2_THT_Pad1.0mm, F.Cu at (-81.2, -103.5)
- added NT440: M2_2, NetTie:NetTie-2_THT_Pad1.0mm, F.Cu at (-105.4, -98.4)
- added NT441: M2_H2, NetTie:NetTie-2_THT_Pad1.0mm, F.Cu at (-81.2, -99.1)
- added NT442: M2_3, NetTie:NetTie-2_THT_Pad1.0mm, F.Cu at (-105.4, -94.0)
- added NT443: M2_H3, NetTie:NetTie-2_THT_Pad1.0mm, F.Cu at (-81.2, -94.6)
- added NT444: M2_4, NetTie:NetTie-2_THT_Pad1.0mm, F.Cu at (-105.4, -89.5)
- added NT445: M2_H4, NetTie:NetTie-2_THT_Pad1.0mm, F.Cu at (-83.8, -90.2)
- added TP76: TestPoint_Small, Connector_Pin:Pin_D1.0mm_L10.0mm, F.Cu at (-111.1, -76.8)
- added TP77: TestPoint_Small, Connector_Pin:Pin_D1.0mm_L10.0mm, F.Cu at (-78.1, -76.8)
- D10, D11, D12, D17, D19, D20, D21, D22: value LED -> 1N4148; footprint LED_THT:LED_D3.0mm_Clear -> Diode_THT:D_DO-35_SOD27_P7.62mm_Horizontal
- J28: renamed from J15; footprint SnapEDA Library:AMPHENOL_L77DFE09S1AMN -> Connector_Dsub:DSUB-9_Female_Horizontal_P2.77x2.84mm_EdgePinOffset4.94mm_Housed_MountingHolesOffset7.48mm
- NT1, NT10, NT100, NT101, NT102, NT103, NT104, NT105, NT106, NT107, NT108, NT109, NT11, NT110, NT111, NT112, NT113, NT114, NT115, NT116, NT117, NT118, NT119, NT12, NT120, NT121, NT122, NT123, NT124, NT125, NT126, NT127, NT128, NT129, NT13, NT130, NT131, NT132, NT133, NT134, NT135, NT14, NT15, NT16, NT17, NT18, NT19, NT2, NT20, NT21, NT22, NT23, NT24, NT25, NT26, NT27, NT28, NT29, NT3, NT30, NT31, NT32, NT33, NT34, NT35, NT36, NT37, NT38, NT39, NT4, NT40, NT41, NT42, NT43, NT432, NT433, NT44, NT45, NT46, NT47, NT48, NT49, NT5, NT50, NT51, NT52, NT53, NT54, NT55, NT56, NT57, NT58, NT59, NT6, NT60, NT61, NT62, NT63, NT64, NT65, NT66, NT67, NT68, NT69, NT7, NT70, NT71, NT72, NT73, NT74, NT75, NT76, NT77, NT78, NT79, NT8, NT80, NT81, NT82, NT83, NT84, NT85, NT86, NT87, NT88, NT89, NT9, NT90, NT91, NT92, NT93, NT94, NT95, NT96, NT97, NT98, NT99: footprint NetTie:NetTie-2_THT_Pad0.3mm -> NetTie:NetTie-2_THT_Pad1.0mm
- NT136: renamed from NT578; footprint NetTie:NetTie-2_THT_Pad0.3mm -> NetTie:NetTie-2_THT_Pad1.0mm
- NT137: renamed from NT136; footprint NetTie:NetTie-2_THT_Pad0.3mm -> NetTie:NetTie-2_THT_Pad1.0mm
- NT138: renamed from NT137; footprint NetTie:NetTie-2_THT_Pad0.3mm -> NetTie:NetTie-2_THT_Pad1.0mm
- NT139: renamed from NT138; footprint NetTie:NetTie-2_THT_Pad0.3mm -> NetTie:NetTie-2_THT_Pad1.0mm
- NT140: renamed from NT139; footprint NetTie:NetTie-2_THT_Pad0.3mm -> NetTie:NetTie-2_THT_Pad1.0mm
- NT141: renamed from NT140; footprint NetTie:NetTie-2_THT_Pad0.3mm -> NetTie:NetTie-2_THT_Pad1.0mm
- NT142: renamed from NT141; footprint NetTie:NetTie-2_THT_Pad0.3mm -> NetTie:NetTie-2_THT_Pad1.0mm
- NT143: renamed from NT142; footprint NetTie:NetTie-2_THT_Pad0.3mm -> NetTie:NetTie-2_THT_Pad1.0mm
- NT144: renamed from NT143; footprint NetTie:NetTie-2_THT_Pad0.3mm -> NetTie:NetTie-2_THT_Pad1.0mm
- NT145: renamed from NT144; footprint NetTie:NetTie-2_THT_Pad0.3mm -> NetTie:NetTie-2_THT_Pad1.0mm
- NT146: renamed from NT145; footprint NetTie:NetTie-2_THT_Pad0.3mm -> NetTie:NetTie-2_THT_Pad1.0mm
- NT147: renamed from NT146; footprint NetTie:NetTie-2_THT_Pad0.3mm -> NetTie:NetTie-2_THT_Pad1.0mm
- NT148: renamed from NT147; footprint NetTie:NetTie-2_THT_Pad0.3mm -> NetTie:NetTie-2_THT_Pad1.0mm
- NT149: renamed from NT148; footprint NetTie:NetTie-2_THT_Pad0.3mm -> NetTie:NetTie-2_THT_Pad1.0mm
- NT150: renamed from NT149; footprint NetTie:NetTie-2_THT_Pad0.3mm -> NetTie:NetTie-2_THT_Pad1.0mm
- NT151: renamed from NT150; footprint NetTie:NetTie-2_THT_Pad0.3mm -> NetTie:NetTie-2_THT_Pad1.0mm
- NT152: renamed from NT151; footprint NetTie:NetTie-2_THT_Pad0.3mm -> NetTie:NetTie-2_THT_Pad1.0mm
- NT153: renamed from NT152; footprint NetTie:NetTie-2_THT_Pad0.3mm -> NetTie:NetTie-2_THT_Pad1.0mm
- NT154: renamed from NT153; footprint NetTie:NetTie-2_THT_Pad0.3mm -> NetTie:NetTie-2_THT_Pad1.0mm
- NT155: renamed from NT154; footprint NetTie:NetTie-2_THT_Pad0.3mm -> NetTie:NetTie-2_THT_Pad1.0mm
- NT156: renamed from NT155; footprint NetTie:NetTie-2_THT_Pad0.3mm -> NetTie:NetTie-2_THT_Pad1.0mm
- NT157: renamed from NT156; footprint NetTie:NetTie-2_THT_Pad0.3mm -> NetTie:NetTie-2_THT_Pad1.0mm
- NT158: renamed from NT157; footprint NetTie:NetTie-2_THT_Pad0.3mm -> NetTie:NetTie-2_THT_Pad1.0mm
- NT159: renamed from NT158; footprint NetTie:NetTie-2_THT_Pad0.3mm -> NetTie:NetTie-2_THT_Pad1.0mm
- NT160: renamed from NT159; footprint NetTie:NetTie-2_THT_Pad0.3mm -> NetTie:NetTie-2_THT_Pad1.0mm
- NT161: renamed from NT160; footprint NetTie:NetTie-2_THT_Pad0.3mm -> NetTie:NetTie-2_THT_Pad1.0mm
- NT162: renamed from NT161; footprint NetTie:NetTie-2_THT_Pad0.3mm -> NetTie:NetTie-2_THT_Pad1.0mm
- NT163: renamed from NT162; footprint NetTie:NetTie-2_THT_Pad0.3mm -> NetTie:NetTie-2_THT_Pad1.0mm
- NT164: renamed from NT163; footprint NetTie:NetTie-2_THT_Pad0.3mm -> NetTie:NetTie-2_THT_Pad1.0mm
- NT165: renamed from NT164; footprint NetTie:NetTie-2_THT_Pad0.3mm -> NetTie:NetTie-2_THT_Pad1.0mm
- NT166: renamed from NT165; footprint NetTie:NetTie-2_THT_Pad0.3mm -> NetTie:NetTie-2_THT_Pad1.0mm
- NT167: renamed from NT579; footprint NetTie:NetTie-2_THT_Pad0.3mm -> NetTie:NetTie-2_THT_Pad1.0mm
- NT168: renamed from NT166; footprint NetTie:NetTie-2_THT_Pad0.3mm -> NetTie:NetTie-2_THT_Pad1.0mm
- NT169: renamed from NT167; footprint NetTie:NetTie-2_THT_Pad0.3mm -> NetTie:NetTie-2_THT_Pad1.0mm
- NT170: renamed from NT168; footprint NetTie:NetTie-2_THT_Pad0.3mm -> NetTie:NetTie-2_THT_Pad1.0mm
- NT171: renamed from NT169; footprint NetTie:NetTie-2_THT_Pad0.3mm -> NetTie:NetTie-2_THT_Pad1.0mm
- NT172: renamed from NT170; footprint NetTie:NetTie-2_THT_Pad0.3mm -> NetTie:NetTie-2_THT_Pad1.0mm
- NT173: renamed from NT171; footprint NetTie:NetTie-2_THT_Pad0.3mm -> NetTie:NetTie-2_THT_Pad1.0mm
- NT174: renamed from NT172; footprint NetTie:NetTie-2_THT_Pad0.3mm -> NetTie:NetTie-2_THT_Pad1.0mm
- NT175: renamed from NT173; footprint NetTie:NetTie-2_THT_Pad0.3mm -> NetTie:NetTie-2_THT_Pad1.0mm
- NT176: renamed from NT174; footprint NetTie:NetTie-2_THT_Pad0.3mm -> NetTie:NetTie-2_THT_Pad1.0mm
- NT177: renamed from NT175; footprint NetTie:NetTie-2_THT_Pad0.3mm -> NetTie:NetTie-2_THT_Pad1.0mm
- NT178: renamed from NT176; footprint NetTie:NetTie-2_THT_Pad0.3mm -> NetTie:NetTie-2_THT_Pad1.0mm
- NT179: renamed from NT177; footprint NetTie:NetTie-2_THT_Pad0.3mm -> NetTie:NetTie-2_THT_Pad1.0mm
- NT180: renamed from NT178; footprint NetTie:NetTie-2_THT_Pad0.3mm -> NetTie:NetTie-2_THT_Pad1.0mm
- NT181: renamed from NT179; footprint NetTie:NetTie-2_THT_Pad0.3mm -> NetTie:NetTie-2_THT_Pad1.0mm
- NT182: renamed from NT180; footprint NetTie:NetTie-2_THT_Pad0.3mm -> NetTie:NetTie-2_THT_Pad1.0mm
- NT183: renamed from NT181; footprint NetTie:NetTie-2_THT_Pad0.3mm -> NetTie:NetTie-2_THT_Pad1.0mm
- NT184: renamed from NT182; footprint NetTie:NetTie-2_THT_Pad0.3mm -> NetTie:NetTie-2_THT_Pad1.0mm
- NT185: renamed from NT183; footprint NetTie:NetTie-2_THT_Pad0.3mm -> NetTie:NetTie-2_THT_Pad1.0mm
- NT186: renamed from NT184; footprint NetTie:NetTie-2_THT_Pad0.3mm -> NetTie:NetTie-2_THT_Pad1.0mm
- NT187: renamed from NT185; footprint NetTie:NetTie-2_THT_Pad0.3mm -> NetTie:NetTie-2_THT_Pad1.0mm
- NT188: renamed from NT186; footprint NetTie:NetTie-2_THT_Pad0.3mm -> NetTie:NetTie-2_THT_Pad1.0mm
- NT189: renamed from NT187; footprint NetTie:NetTie-2_THT_Pad0.3mm -> NetTie:NetTie-2_THT_Pad1.0mm
- NT190: renamed from NT188; footprint NetTie:NetTie-2_THT_Pad0.3mm -> NetTie:NetTie-2_THT_Pad1.0mm
- NT191: renamed from NT189; footprint NetTie:NetTie-2_THT_Pad0.3mm -> NetTie:NetTie-2_THT_Pad1.0mm
- NT192: renamed from NT190; footprint NetTie:NetTie-2_THT_Pad0.3mm -> NetTie:NetTie-2_THT_Pad1.0mm
- NT193: renamed from NT191; footprint NetTie:NetTie-2_THT_Pad0.3mm -> NetTie:NetTie-2_THT_Pad1.0mm
- NT194: renamed from NT192; footprint NetTie:NetTie-2_THT_Pad0.3mm -> NetTie:NetTie-2_THT_Pad1.0mm
- NT195: renamed from NT193; footprint NetTie:NetTie-2_THT_Pad0.3mm -> NetTie:NetTie-2_THT_Pad1.0mm
- NT196: renamed from NT194; footprint NetTie:NetTie-2_THT_Pad0.3mm -> NetTie:NetTie-2_THT_Pad1.0mm
- NT197: renamed from NT195; footprint NetTie:NetTie-2_THT_Pad0.3mm -> NetTie:NetTie-2_THT_Pad1.0mm
- NT198: renamed from NT580; footprint NetTie:NetTie-2_THT_Pad0.3mm -> NetTie:NetTie-2_THT_Pad1.0mm
- NT199: renamed from NT196; footprint NetTie:NetTie-2_THT_Pad0.3mm -> NetTie:NetTie-2_THT_Pad1.0mm
- NT200: renamed from NT197; footprint NetTie:NetTie-2_THT_Pad0.3mm -> NetTie:NetTie-2_THT_Pad1.0mm
- NT201: renamed from NT198; footprint NetTie:NetTie-2_THT_Pad0.3mm -> NetTie:NetTie-2_THT_Pad1.0mm
- NT202: renamed from NT199; footprint NetTie:NetTie-2_THT_Pad0.3mm -> NetTie:NetTie-2_THT_Pad1.0mm
- NT203: renamed from NT200; footprint NetTie:NetTie-2_THT_Pad0.3mm -> NetTie:NetTie-2_THT_Pad1.0mm
- NT204: renamed from NT201; footprint NetTie:NetTie-2_THT_Pad0.3mm -> NetTie:NetTie-2_THT_Pad1.0mm
- NT205: renamed from NT202; footprint NetTie:NetTie-2_THT_Pad0.3mm -> NetTie:NetTie-2_THT_Pad1.0mm
- NT206: renamed from NT203; footprint NetTie:NetTie-2_THT_Pad0.3mm -> NetTie:NetTie-2_THT_Pad1.0mm
- NT207: renamed from NT204; footprint NetTie:NetTie-2_THT_Pad0.3mm -> NetTie:NetTie-2_THT_Pad1.0mm
- NT208: renamed from NT205; footprint NetTie:NetTie-2_THT_Pad0.3mm -> NetTie:NetTie-2_THT_Pad1.0mm
- NT209: renamed from NT206; footprint NetTie:NetTie-2_THT_Pad0.3mm -> NetTie:NetTie-2_THT_Pad1.0mm
- NT210: renamed from NT207; footprint NetTie:NetTie-2_THT_Pad0.3mm -> NetTie:NetTie-2_THT_Pad1.0mm
- NT211: renamed from NT208; footprint NetTie:NetTie-2_THT_Pad0.3mm -> NetTie:NetTie-2_THT_Pad1.0mm
- NT212: renamed from NT209; footprint NetTie:NetTie-2_THT_Pad0.3mm -> NetTie:NetTie-2_THT_Pad1.0mm
- NT213: renamed from NT210; footprint NetTie:NetTie-2_THT_Pad0.3mm -> NetTie:NetTie-2_THT_Pad1.0mm
- NT214: renamed from NT211; footprint NetTie:NetTie-2_THT_Pad0.3mm -> NetTie:NetTie-2_THT_Pad1.0mm
- NT215: renamed from NT212; footprint NetTie:NetTie-2_THT_Pad0.3mm -> NetTie:NetTie-2_THT_Pad1.0mm
- NT216: renamed from NT213; footprint NetTie:NetTie-2_THT_Pad0.3mm -> NetTie:NetTie-2_THT_Pad1.0mm
- NT217: renamed from NT214; footprint NetTie:NetTie-2_THT_Pad0.3mm -> NetTie:NetTie-2_THT_Pad1.0mm
- NT218: renamed from NT215; footprint NetTie:NetTie-2_THT_Pad0.3mm -> NetTie:NetTie-2_THT_Pad1.0mm
- NT219: renamed from NT216; footprint NetTie:NetTie-2_THT_Pad0.3mm -> NetTie:NetTie-2_THT_Pad1.0mm
- NT220: renamed from NT217; footprint NetTie:NetTie-2_THT_Pad0.3mm -> NetTie:NetTie-2_THT_Pad1.0mm
- NT221: renamed from NT218; footprint NetTie:NetTie-2_THT_Pad0.3mm -> NetTie:NetTie-2_THT_Pad1.0mm
- NT222: renamed from NT219; footprint NetTie:NetTie-2_THT_Pad0.3mm -> NetTie:NetTie-2_THT_Pad1.0mm
- NT223: renamed from NT220; footprint NetTie:NetTie-2_THT_Pad0.3mm -> NetTie:NetTie-2_THT_Pad1.0mm
- NT224: renamed from NT221; footprint NetTie:NetTie-2_THT_Pad0.3mm -> NetTie:NetTie-2_THT_Pad1.0mm
- NT225: renamed from NT222; footprint NetTie:NetTie-2_THT_Pad0.3mm -> NetTie:NetTie-2_THT_Pad1.0mm
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- renumbered D5 to D1, D26 to D13, D31 to D14, D32 to D15, D33 to D16, D36 to D18, D6 to D2, D43 to D25, D44 to D26, D47 to D29, D7 to D3, D87 to D30, D88 to D31, D89 to D32, D90 to D33, D48 to D34, D49 to D35, D50 to D36, D55 to D37, D56 to D38, D57 to D39, D8 to D4, D58 to D40, D63 to D41, D64 to D42, D65 to D43, D66 to D44, D68 to D45, D73 to D46, D74 to D47, D75 to D48, D76 to D49, D13 to D5, D81 to D50, D82 to D51, D83 to D52, D84 to D53, D86 to D54, D14 to D6, D15 to D7, D16 to D8, D18 to D9, J22 to J10, J23 to J11, J24 to J12, J25 to J13, J26 to J14, J27 to J15, J28 to J16, J5 to J17, J6 to J18, J7 to J19, J8 to J20, J9 to J21, J10 to J22, J17 to J23, J12 to J24, J13 to J25, J11 to J26, J14 to J27, J33 to J29, J29 to J30, J30 to J31, J31 to J32, J32 to J33, J16 to J5, J18 to J6, J19 to J7, J20 to J8, J21 to J9, K5 to K1, K14 to K10, K15 to K11, K16 to K12, K17 to K13, K18 to K14, K19 to K15, K20 to K16, K21 to K17, K22 to K18, K23 to K19, K6 to K2, K1 to K20, K3 to K21, K2 to K22, K4 to K23, K7 to K3, K8 to K4, K9 to K5, K10 to K6, K11 to K7, K12 to K8, K13 to K9, Q55 to Q19, Q19 to Q20, Q20 to Q21, Q56 to Q22, Q21 to Q23, Q57 to Q24, Q22 to Q25, Q35 to Q38, Q36 to Q39, Q37 to Q40, Q38 to Q41, Q39 to Q42, Q40 to Q43, Q41 to Q44, Q42 to Q45, Q43 to Q46, Q44 to Q47, Q45 to Q48, Q46 to Q49, Q47 to Q50, Q48 to Q51, Q49 to Q52, Q50 to Q53, Q51 to Q54, Q52 to Q55, Q53 to Q56, Q54 to Q57, R5 to R1, R132 to R101, R20 to R11, R21 to R12, R22 to R13, R23 to R14, R25 to R16, R31 to R18, R32 to R19, R33 to R20, R34 to R21, R39 to R22, R40 to R23, R41 to R24, R42 to R25, R44 to R26, R45 to R27, R46 to R28, R133 to R31, R49 to R33, R50 to R34, R134 to R35, R52 to R36, R54 to R38, R8 to R4, R135 to R40, R56 to R41, R57 to R42, R58 to R43, R59 to R44, R60 to R45, R61 to R46, R62 to R47, R63 to R48, R64 to R49, R13 to R5, R65 to R50, R66 to R51, R67 to R52, R68 to R53, R69 to R54, R70 to R55, R71 to R56, R72 to R57, R73 to R58, R74 to R59, R14 to R6, R75 to R60, R76 to R61, R77 to R62, R78 to R63, R79 to R64, R80 to R65, R136 to R66, R137 to R67, R81 to R68, R82 to R69, R15 to R7, R83 to R70, R84 to R71, R85 to R72, R86 to R73, R87 to R74, R88 to R75, R89 to R76, R90 to R77, R91 to R78, R92 to R79, R16 to R8, R93 to R80, R94 to R81, R95 to R82, R96 to R83, R101 to R84, R102 to R85, R103 to R86, R104 to R87, R109 to R88, R110 to R89, R18 to R9, R111 to R90, R112 to R91, R114 to R92, R119 to R93, R120 to R94, R121 to R95, R122 to R96, R128 to R98, R129 to R99, U4 to U3, U5 to U4, U3 to U5
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Connections:
- net PM3_IO28 renamed PM2_IO28
- net PM3_IO8 renamed PM2_IO8
- net PM3_IO9 renamed PM2_IO9
- BZ1 pad 1: VCC -> PWR_5V
- C1 pad 1: VCC -> PWR_5V
- C14 pad 1: VCC -> PWR_5V
- C15 pad 1: VCC -> PWR_5V
- C16 pad 1: VCC -> PWR_5V
- C17 pad 1: VCC -> PWR_5V
- C2 pad 1: VCC -> PWR_5V
- D1 pad 1: VCC -> PWR_5V
- D10 pad 1: Net-(D10-Pad1) -> PWR_5V
- D10 pad 2: VCC -> Net-(D10-Pad2)
- D11 pad 1: Net-(D11-Pad1) -> PWR_5V
- D11 pad 2: VCC -> Net-(D11-Pad2)
- D12 pad 1: Net-(D12-Pad1) -> PWR_5V
- D12 pad 2: VCC -> Net-(D12-Pad2)
- D13 pad 1: VCC -> PWR_5V
- D14 pad 1: VCC -> PWR_5V
- D15 pad 1: VCC -> PWR_5V
- D16 pad 1: VCC -> PWR_5V
- D17 pad 1: Net-(D17-Pad1) -> PWR_5V
- D17 pad 2: VCC -> Net-(D17-Pad2)
- D18 pad 1: VCC -> PWR_5V
- D19 pad 1: Net-(D19-Pad1) -> MSR_3V3
- D19 pad 2: VCC -> ADC0
- D2 pad 1: VCC -> PWR_5V
- D2 pad 2: Net-(D6-Pad2) -> Net-(D2-Pad2)
- D20 pad 1: Net-(D20-Pad1) -> ADC0
- D20 pad 2: VCC -> GND
- D21 pad 1: Net-(D21-Pad1) -> MSR_3V3
- D21 pad 2: VCC -> ADC1
- D22 pad 1: Net-(D22-Pad1) -> ADC1
- D22 pad 2: VCC -> GND
- D23 pad 1: VCC -> Net-(D23-Pad1)
- D23 pad 2: Net-(D23-Pad2) -> GND
- D25 pad 1: VCC -> PWR_5V
- D26 pad 1: VCC -> PWR_5V
- D29 pad 1: VCC -> PWR_5V
- D3 pad 1: VCC -> PWR_5V
- D3 pad 2: Net-(D7-Pad2) (its old number) -> Net-(D3-Pad2)
- D34 pad 1: VCC -> PWR_5V
- D36 pad 2: VCC -> PWR_5V
- D37 pad 1: VCC -> PWR_5V
- D37 pad 2: Net-(D55-Pad2) -> Net-(D37-Pad2)
- D38 pad 1: VCC -> PWR_5V
- D39 pad 1: VCC -> PWR_5V
- D4 pad 1: VCC -> PWR_5V
- D40 pad 1: VCC -> PWR_5V
- D40 pad 2: Net-(D58-Pad2) -> Net-(D40-Pad2)
- D41 pad 1: VCC -> PWR_5V
- D42 pad 1: VCC -> PWR_5V
- D43 pad 1: VCC -> PWR_5V
- D44 pad 1: VCC -> PWR_5V
- D45 pad 1: VCC -> PWR_5V
- D46 pad 1: VCC -> PWR_5V
- D47 pad 1: VCC -> PWR_5V
- D48 pad 1: VCC -> PWR_5V
- D49 pad 1: VCC -> PWR_5V
- D5 pad 1: VCC -> PWR_5V
- D50 pad 1: VCC -> PWR_5V
- D51 pad 1: VCC -> PWR_5V
- D52 pad 1: VCC -> PWR_5V
- D53 pad 1: VCC -> PWR_5V
- D54 pad 1: VCC -> PWR_5V
- D6 pad 1: VCC -> PWR_5V
- D6 pad 2: Net-(D14-Pad2) (its old number) -> Net-(D6-Pad2)
- D7 pad 1: VCC -> PWR_5V
- D8 pad 1: VCC -> PWR_5V
- D9 pad 1: VCC -> PWR_5V
- D9 pad 2: Net-(D18-Pad2) (its old number) -> Net-(D9-Pad2)
- F1 pad P$2: VCC -> PWR_5V
- J11 pad 1: /Communication/M3_LV1 -> /Communication/M2_LV1
- J11 pad 2: /Communication/M3_LV2 -> /Communication/M2_LV2
- J11 pad 5: /Communication/M3_LV3 -> /Communication/M2_LV3
- J11 pad 6: /Communication/M3_LV4 -> /Communication/M2_LV4
- J12 pad 1: /Communication/M3_HV1 -> /Communication/M2_HV1
- J12 pad 2: /Communication/M3_HV2 -> /Communication/M2_HV2
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Routing:
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Other:
- board size 396.5 x 196.6 mm -> 412 x 195.1 mm

Commit message: backup 1 bank done
Parts:
- removed D1, D10, D11, D12, D13, D14, D15, D16, D17, D18, D2, D25, D26, D29, D3, D37, D38, D39, D4, D40, D41, D42, D43, D44, D45, D46, D47, D48, D49, D5, D50, D51, D52, D53, D54, D6, D7, D8, D9: 1N4148, Diode_THT:D_DO-35_SOD27_P7.62mm_Horizontal
- removed NT526: NT24_CL, NetTie:NetTie-2_THT_Pad1.0mm
- removed NT527: NT25_CL, NetTie:NetTie-2_THT_Pad1.0mm
- removed NT528: NT26_CL, NetTie:NetTie-2_THT_Pad1.0mm
- removed NT529: NT27_CL, NetTie:NetTie-2_THT_Pad1.0mm
- removed NT530: NT24_D, NetTie:NetTie-2_THT_Pad1.0mm
- removed NT531: NT25_D, NetTie:NetTie-2_THT_Pad1.0mm
- removed NT532: NT26_D, NetTie:NetTie-2_THT_Pad1.0mm
- removed NT533: NT27_D, NetTie:NetTie-2_THT_Pad1.0mm
- removed NT534, NT537: NT2S_RL, NetTie:NetTie-2_THT_Pad1.0mm
- removed NT535: NT2S_CH, NetTie:NetTie-2_THT_Pad1.0mm
- removed NT536: NT2S_NH, NetTie:NetTie-2_THT_Pad1.0mm
- removed NT538: NT2S_CL, NetTie:NetTie-2_THT_Pad1.0mm
- removed NT539: NT2S_L1, NetTie:NetTie-2_THT_Pad1.0mm
- removed NT540: NT2S_D, NetTie:NetTie-2_THT_Pad1.0mm
- removed NT541: NT30_H, NetTie:NetTie-2_THT_Pad1.0mm
- removed NT542: NT31_H, NetTie:NetTie-2_THT_Pad1.0mm
- removed NT543: NT32_H, NetTie:NetTie-2_THT_Pad1.0mm
- removed NT544: NT33_H, NetTie:NetTie-2_THT_Pad1.0mm
- removed NT545: NT30_CH, NetTie:NetTie-2_THT_Pad1.0mm
- removed NT546: NT31_CH, NetTie:NetTie-2_THT_Pad1.0mm
- removed NT547: NT32_CH, NetTie:NetTie-2_THT_Pad1.0mm
- removed NT548: NT33_CH, NetTie:NetTie-2_THT_Pad1.0mm
- removed NT549: NT30_L, NetTie:NetTie-2_THT_Pad1.0mm
- removed NT550: NT31_L, NetTie:NetTie-2_THT_Pad1.0mm
- removed NT551: NT32_L, NetTie:NetTie-2_THT_Pad1.0mm
- removed NT552: NT33_L, NetTie:NetTie-2_THT_Pad1.0mm
- removed NT553: NT30_CL, NetTie:NetTie-2_THT_Pad1.0mm
- removed NT554: NT31_CL, NetTie:NetTie-2_THT_Pad1.0mm
- removed NT555: NT32_CL, NetTie:NetTie-2_THT_Pad1.0mm
- removed NT556: NT33_CL, NetTie:NetTie-2_THT_Pad1.0mm
- removed NT557: NT30_D, NetTie:NetTie-2_THT_Pad1.0mm
- removed NT558: NT31_D, NetTie:NetTie-2_THT_Pad1.0mm
- removed NT559: NT32_D, NetTie:NetTie-2_THT_Pad1.0mm
- removed NT560: NT33_D, NetTie:NetTie-2_THT_Pad1.0mm
- removed NT561: NT34_H, NetTie:NetTie-2_THT_Pad1.0mm
- removed NT562: NT35_H, NetTie:NetTie-2_THT_Pad1.0mm
- removed NT563: NT36_H, NetTie:NetTie-2_THT_Pad1.0mm
- removed NT564: NT37_H, NetTie:NetTie-2_THT_Pad1.0mm
- removed NT565: NT34_CH, NetTie:NetTie-2_THT_Pad1.0mm
- removed NT566: NT35_CH, NetTie:NetTie-2_THT_Pad1.0mm
- removed NT567: NT36_CH, NetTie:NetTie-2_THT_Pad1.0mm
- removed NT568: NT37_CH, NetTie:NetTie-2_THT_Pad1.0mm
- removed NT569: NT34_L, NetTie:NetTie-2_THT_Pad1.0mm
- removed NT570: NT35_L, NetTie:NetTie-2_THT_Pad1.0mm
- removed NT571: NT36_L, NetTie:NetTie-2_THT_Pad1.0mm
- removed NT572: NT37_L, NetTie:NetTie-2_THT_Pad1.0mm
- removed NT573: NT34_CL, NetTie:NetTie-2_THT_Pad1.0mm
- removed NT574: NT35_CL, NetTie:NetTie-2_THT_Pad1.0mm
- removed NT575: NT36_CL, NetTie:NetTie-2_THT_Pad1.0mm
- removed NT576: NT37_CL, NetTie:NetTie-2_THT_Pad1.0mm
- removed NT577: NT34_D, NetTie:NetTie-2_THT_Pad1.0mm
- removed NT578: NT35_D, NetTie:NetTie-2_THT_Pad1.0mm
- removed NT579: NT36_D, NetTie:NetTie-2_THT_Pad1.0mm
- removed NT580: NT37_D, NetTie:NetTie-2_THT_Pad1.0mm
- removed NT581, NT584: NT3S_RL, NetTie:NetTie-2_THT_Pad1.0mm
- removed NT582: NT3S_CH, NetTie:NetTie-2_THT_Pad1.0mm
- removed NT583: NT3S_NH, NetTie:NetTie-2_THT_Pad1.0mm
- removed NT585: NT3S_CL, NetTie:NetTie-2_THT_Pad1.0mm
- removed NT586: NT3S_L1, NetTie:NetTie-2_THT_Pad1.0mm
- removed NT587: NT3S_D, NetTie:NetTie-2_THT_Pad1.0mm
- removed Q1, Q10, Q11, Q12, Q13, Q14, Q15, Q16, Q17, Q18, Q2, Q20, Q21, Q23, Q25, Q3, Q38, Q39, Q4, Q40, Q41, Q42, Q43, Q44, Q45, Q46, Q47, Q48, Q49, Q5, Q50, Q51, Q52, Q53, Q54, Q55, Q56, Q57, Q6, Q7, Q8, Q9: 2N2222, Package_TO_SOT_THT:TO-92_Inline
- removed R100, R101, R18, R19, R2, R20, R21, R22, R23, R24, R25, R26, R3, R33, R34, R38, R4, R41, R5, R6, R7, R70, R72, R8, R84, R85, R86, R87, R88, R89, R9, R90, R91, R92, R93, R94, R95, R96, R97, R98, R99: 10K, Resistor_THT:R_Axial_DIN0309_L9.0mm_D3.2mm_P12.70mm_Horizontal
- removed R15: 4.7K, Package_TO_SOT_SMD:SOT-23-8
- removed TP127: NT35_HH, Connector_Pin:Pin_D1.0mm_L10.0mm
- removed TP128: NT36_HH, Connector_Pin:Pin_D1.0mm_L10.0mm
- removed TP129: NT37_HH, Connector_Pin:Pin_D1.0mm_L10.0mm
- removed TP130: NT34_LL, Connector_Pin:Pin_D1.0mm_L10.0mm
- removed TP131: NT35_LL, Connector_Pin:Pin_D1.0mm_L10.0mm
- removed TP132: NT36_LL, Connector_Pin:Pin_D1.0mm_L10.0mm
- removed TP133: NT37_LL, Connector_Pin:Pin_D1.0mm_L10.0mm
- added REF**: DIN41612_R_3x32_Male_Horizontal_THT, Connector_DIN:DIN41612_R_3x32_Male_Horizontal_THT, F.Cu at (372.3, 47.7)
- added TP89: NT20_HH, Connector_Pin:Pin_D0.9mm_L10.0mm_W2.4mm_FlatFork, F.Cu at (332.7, -67.6)
- added TP90: NT21_HH, Connector_Pin:Pin_D0.9mm_L10.0mm_W2.4mm_FlatFork, F.Cu at (351.8, -68.2)
- added TP91: NT22_HH, Connector_Pin:Pin_D0.9mm_L10.0mm_W2.4mm_FlatFork, F.Cu at (370.2, -68.2)
- added TP93: NT23_HH, Connector_Pin:Pin_D0.9mm_L10.0mm_W2.4mm_FlatFork, F.Cu at (331.4, -51.7)
- added TP95: NT20_LL, Connector_Pin:Pin_D0.9mm_L10.0mm_W2.4mm_FlatFork, F.Cu at (334.6, -60.0)
- added TP96: NT21_LL, Connector_Pin:Pin_D0.9mm_L10.0mm_W2.4mm_FlatFork, F.Cu at (353.0, -59.3)
- added TP99: NT22_LL, Connector_Pin:Pin_D0.9mm_L10.0mm_W2.4mm_FlatFork, F.Cu at (373.4, -59.3)
- added U13: ULN2003A, Package_DIP:DIP-16_W7.62mm_LongPads, F.Cu at (399.6, 244.1)
- added U14: ULN2003A, Package_DIP:DIP-16_W7.62mm_LongPads, F.Cu at (399.6, 216.9)
- added U15: ULN2003A, Package_DIP:DIP-16_W7.62mm_LongPads, F.Cu at (422.1, 232.9)
- added U16: ULN2003A, Package_DIP:DIP-16_W7.62mm_LongPads, F.Cu at (421.9, 204.5)
- added U17: ULN2003A, Package_DIP:DIP-16_W7.62mm_LongPads, F.Cu at (399.5, 191.8)
- added U18: ULN2003A, Package_DIP:DIP-16_W7.62mm_LongPads, F.Cu at (414.5, 156.2)
- NT1: value NT10_H -> NT10_CH; footprint NetTie:NetTie-2_THT_Pad1.0mm -> NetTie:NetTie-2_Front1.0mm
- NT10: value NT11_L -> NT15_CH; footprint NetTie:NetTie-2_THT_Pad1.0mm -> NetTie:NetTie-2_Front1.0mm
- NT100, NT101, NT102, NT103, NT104, NT105, NT106, NT107, NT108, NT109, NT110, NT111, NT112, NT113, NT114, NT115, NT116, NT117, NT118, NT119, NT120, NT121, NT122, NT123, NT124, NT125, NT126, NT127, NT128, NT129, NT130, NT131, NT132, NT133, NT134, NT135, NT136, NT137, NT138, NT139, NT140, NT141, NT142, NT143, NT144, NT145, NT146, NT147, NT148, NT149, NT150, NT151, NT152, NT153, NT154, NT155, NT156, NT157, NT158, NT159, NT160, NT161, NT162, NT163, NT164, NT165, NT166, NT167, NT168, NT169, NT170, NT171, NT172, NT173, NT174, NT175, NT176, NT177, NT178, NT179, NT180, NT181, NT182, NT183, NT184, NT185, NT186, NT187, NT188, NT189, NT190, NT191, NT192, NT193, NT194, NT195, NT196, NT197, NT198, NT199, NT200, NT201, NT202, NT203, NT204, NT205, NT206, NT207, NT208, NT209, NT210, NT211, NT212, NT213, NT214, NT215, NT216, NT217, NT218, NT219, NT220, NT221, NT222, NT223, NT224, NT225, NT226, NT227, NT228, NT229, NT230, NT231, NT232, NT233, NT234, NT235, NT236, NT237, NT238, NT239, NT240, NT241, NT242, NT243, NT244, NT245, NT246, NT247, NT248, NT249, NT250, NT251, NT252, NT253, NT254, NT255, NT256, NT257, NT258, NT259, NT260, NT261, NT262, NT263, NT264, NT265, NT266, NT267, NT268, NT269, NT270, NT271, NT272, NT273, NT274, NT275, NT276, NT277, NT278, NT279, NT280, NT281, NT282, NT283, NT284, NT285, NT286, NT287, NT288, NT289, NT290, NT291, NT292, NT293, NT295, NT296, NT297, NT298, NT299, NT300, NT301, NT302, NT303, NT304, NT305, NT306, NT307, NT308, NT309, NT310, NT311, NT312, NT313, NT314, NT315, NT316, NT317, NT318, NT319, NT320, NT321, NT322, NT323, NT324, NT325, NT326, NT327, NT328, NT329, NT330, NT331, NT332, NT333, NT334, NT335, NT336, NT337, NT338, NT339, NT340, NT341, NT342, NT343, NT344, NT345, NT346, NT347, NT348, NT396, NT397, NT398, NT399, NT400, NT401, NT402, NT403, NT404, NT405, NT406, NT407, NT408, NT409, NT412, NT413, NT414, NT415, NT416, NT417, NT418, NT420, NT422, NT423, NT424, NT425, NT426, NT427, NT428, NT429, NT430, NT431, NT432, NT433, NT434, NT435, NT436, NT437, NT438, NT439, NT440, NT441, NT442, NT443, NT444, NT445, NT446, NT447, NT448, NT449, NT450, NT451, NT452, NT453, NT454, NT455, NT456, NT457, NT458, NT459, NT460, NT461, NT462, NT463, NT464, NT465, NT466, NT467, NT468, NT469, NT470, NT471, NT472, NT473, NT474, NT475, NT476, NT477, NT478, NT479, NT48, NT480, NT481, NT482, NT483, NT484, NT485, NT486, NT487, NT488, NT489, NT49, NT490, NT491, NT492, NT493, NT50, NT51, NT52, NT53, NT54, NT55, NT56, NT57, NT58, NT59, NT60, NT61, NT62, NT63, NT64, NT65, NT66, NT67, NT68, NT69, NT70, NT71, NT72, NT73, NT74, NT75, NT76, NT77, NT78, NT79, NT80, NT81, NT82, NT83, NT84, NT85, NT86, NT87, NT88, NT89, NT90, NT91, NT92, NT93, NT94, NT95, NT96, NT97, NT98, NT99: footprint NetTie:NetTie-2_THT_Pad1.0mm -> NetTie:NetTie-2_Front1.0mm
- NT11: value NT12_L -> NT16_CH; footprint NetTie:NetTie-2_THT_Pad1.0mm -> NetTie:NetTie-2_Front1.0mm
- NT12: value NT13_L -> NT17_CH; footprint NetTie:NetTie-2_THT_Pad1.0mm -> NetTie:NetTie-2_Front1.0mm
- NT13: value NT10_CL -> NT14_CL; footprint NetTie:NetTie-2_THT_Pad1.0mm -> NetTie:NetTie-2_Front1.0mm
- NT14: value NT11_CL -> NT15_CL; footprint NetTie:NetTie-2_THT_Pad1.0mm -> NetTie:NetTie-2_Front1.0mm
- NT15: value NT12_CL -> NT16_CL; footprint NetTie:NetTie-2_THT_Pad1.0mm -> NetTie:NetTie-2_Front1.0mm
- NT16: value NT13_CL -> NT17_CL; footprint NetTie:NetTie-2_THT_Pad1.0mm -> NetTie:NetTie-2_Front1.0mm
- NT17: value NT10_D -> NT1S_RL; footprint NetTie:NetTie-2_THT_Pad1.0mm -> NetTie:NetTie-2_Front1.0mm
- NT18: value NT11_D -> NT1S_CH; footprint NetTie:NetTie-2_THT_Pad1.0mm -> NetTie:NetTie-2_Front1.0mm
- NT19: value NT12_D -> NT1S_NH; footprint NetTie:NetTie-2_THT_Pad1.0mm -> NetTie:NetTie-2_Front1.0mm
- NT2: value NT11_H -> NT11_CH; footprint NetTie:NetTie-2_THT_Pad1.0mm -> NetTie:NetTie-2_Front1.0mm
- NT20: value NT13_D -> NT1S_RL; footprint NetTie:NetTie-2_THT_Pad1.0mm -> NetTie:NetTie-2_Front1.0mm
- NT21: value NT14_H -> NT1S_CL; footprint NetTie:NetTie-2_THT_Pad1.0mm -> NetTie:NetTie-2_Front1.0mm
- NT22: value NT15_H -> NT1S_L1; footprint NetTie:NetTie-2_THT_Pad1.0mm -> NetTie:NetTie-2_Front1.0mm
- NT23: value NT16_H -> NT40_CH; footprint NetTie:NetTie-2_THT_Pad1.0mm -> NetTie:NetTie-2_Front1.0mm
- NT24: value NT17_H -> NT41_CH; footprint NetTie:NetTie-2_THT_Pad1.0mm -> NetTie:NetTie-2_Front1.0mm
- NT25: value NT14_CH -> NT42_CH; footprint NetTie:NetTie-2_THT_Pad1.0mm -> NetTie:NetTie-2_Front1.0mm
- NT26: value NT15_CH -> NT43_CH; footprint NetTie:NetTie-2_THT_Pad1.0mm -> NetTie:NetTie-2_Front1.0mm
- NT27: value NT16_CH -> NT40_CL; footprint NetTie:NetTie-2_THT_Pad1.0mm -> NetTie:NetTie-2_Front1.0mm
- NT28: value NT17_CH -> NT41_CL; footprint NetTie:NetTie-2_THT_Pad1.0mm -> NetTie:NetTie-2_Front1.0mm
- NT29: value NT14_L -> NT42_CL; footprint NetTie:NetTie-2_THT_Pad1.0mm -> NetTie:NetTie-2_Front1.0mm
- NT294: footprint Package_TO_SOT_SMD:SOT-23-8 -> NetTie:NetTie-2_Front1.0mm
- NT3: value NT12_H -> NT12_CH; footprint NetTie:NetTie-2_THT_Pad1.0mm -> NetTie:NetTie-2_Front1.0mm
- NT30: value NT15_L -> NT43_CL; footprint NetTie:NetTie-2_THT_Pad1.0mm -> NetTie:NetTie-2_Front1.0mm
- NT31: value NT16_L -> NT44_CH; footprint NetTie:NetTie-2_THT_Pad1.0mm -> NetTie:NetTie-2_Front1.0mm
- NT32: value NT17_L -> NT45_CH; footprint NetTie:NetTie-2_THT_Pad1.0mm -> NetTie:NetTie-2_Front1.0mm
- NT33: value NT14_CL -> NT46_CH; footprint NetTie:NetTie-2_THT_Pad1.0mm -> NetTie:NetTie-2_Front1.0mm
- NT34: value NT15_CL -> NT47_CH; footprint NetTie:NetTie-2_THT_Pad1.0mm -> NetTie:NetTie-2_Front1.0mm
- NT349: value NT40_H -> NT23_CH; footprint NetTie:NetTie-2_THT_Pad1.0mm -> NetTie:NetTie-2_Front1.0mm
- NT35: value NT16_CL -> NT44_CL; footprint NetTie:NetTie-2_THT_Pad1.0mm -> NetTie:NetTie-2_Front1.0mm
- NT350: value NT41_H -> NT20_CL; footprint NetTie:NetTie-2_THT_Pad1.0mm -> NetTie:NetTie-2_Front1.0mm
- NT351: value NT42_H -> NT21_CL; footprint NetTie:NetTie-2_THT_Pad1.0mm -> NetTie:NetTie-2_Front1.0mm
- NT352: value NT43_H -> NT22_CL; footprint NetTie:NetTie-2_THT_Pad1.0mm -> NetTie:NetTie-2_Front1.0mm
- NT353: value NT40_CH -> NT23_CL; footprint NetTie:NetTie-2_THT_Pad1.0mm -> NetTie:NetTie-2_Front1.0mm
- NT354: value NT41_CH -> NT24_CH; footprint NetTie:NetTie-2_THT_Pad1.0mm -> NetTie:NetTie-2_Front1.0mm
- NT355: value NT42_CH -> NT25_CH; footprint NetTie:NetTie-2_THT_Pad1.0mm -> NetTie:NetTie-2_Front1.0mm
- NT356: value NT43_CH -> NT26_CH; footprint NetTie:NetTie-2_THT_Pad1.0mm -> NetTie:NetTie-2_Front1.0mm
- NT357: value NT40_L -> NT27_CH; footprint NetTie:NetTie-2_THT_Pad1.0mm -> NetTie:NetTie-2_Front1.0mm
- NT358: value NT41_L -> NT24_CL; footprint NetTie:NetTie-2_THT_Pad1.0mm -> NetTie:NetTie-2_Front1.0mm
- NT359: value NT42_L -> NT25_CL; footprint NetTie:NetTie-2_THT_Pad1.0mm -> NetTie:NetTie-2_Front1.0mm
- NT36: value NT17_CL -> NT45_CL; footprint NetTie:NetTie-2_THT_Pad1.0mm -> NetTie:NetTie-2_Front1.0mm
- NT360: value NT43_L -> NT26_CL; footprint NetTie:NetTie-2_THT_Pad1.0mm -> NetTie:NetTie-2_Front1.0mm
- NT361: value NT40_CL -> NT27_CL; footprint NetTie:NetTie-2_THT_Pad1.0mm -> NetTie:NetTie-2_Front1.0mm
- NT362: value NT41_CL -> NT2S_RL; footprint NetTie:NetTie-2_THT_Pad1.0mm -> NetTie:NetTie-2_Front1.0mm
- NT363: value NT42_CL -> NT2S_CH; footprint NetTie:NetTie-2_THT_Pad1.0mm -> NetTie:NetTie-2_Front1.0mm
- NT364: value NT43_CL -> NT2S_NH; footprint NetTie:NetTie-2_THT_Pad1.0mm -> NetTie:NetTie-2_Front1.0mm
- NT365: value NT40_D -> NT2S_RL; footprint NetTie:NetTie-2_THT_Pad1.0mm -> NetTie:NetTie-2_Front1.0mm
- NT366: value NT41_D -> NT2S_CL; footprint NetTie:NetTie-2_THT_Pad1.0mm -> NetTie:NetTie-2_Front1.0mm
- NT367: value NT42_D -> NT2S_L1; footprint NetTie:NetTie-2_THT_Pad1.0mm -> NetTie:NetTie-2_Front1.0mm
- NT368: value NT43_D -> NT30_CH; footprint NetTie:NetTie-2_THT_Pad1.0mm -> NetTie:NetTie-2_Front1.0mm
- NT369: value NT44_H -> NT31_CH; footprint NetTie:NetTie-2_THT_Pad1.0mm -> NetTie:NetTie-2_Front1.0mm
- NT37: value NT14_D -> NT46_CL; footprint NetTie:NetTie-2_THT_Pad1.0mm -> NetTie:NetTie-2_Front1.0mm
- NT370: value NT45_H -> NT32_CH; footprint NetTie:NetTie-2_THT_Pad1.0mm -> NetTie:NetTie-2_Front1.0mm
- NT371: value NT46_H -> NT33_CH; footprint NetTie:NetTie-2_THT_Pad1.0mm -> NetTie:NetTie-2_Front1.0mm
- NT372: value NT47_H -> NT30_CL; footprint NetTie:NetTie-2_THT_Pad1.0mm -> NetTie:NetTie-2_Front1.0mm
- NT373: value NT44_CH -> NT31_CL; footprint NetTie:NetTie-2_THT_Pad1.0mm -> NetTie:NetTie-2_Front1.0mm
- NT374: value NT45_CH -> NT32_CL; footprint NetTie:NetTie-2_THT_Pad1.0mm -> NetTie:NetTie-2_Front1.0mm
- NT375: value NT46_CH -> NT33_CL; footprint NetTie:NetTie-2_THT_Pad1.0mm -> NetTie:NetTie-2_Front1.0mm
- NT376: value NT47_CH -> NT34_CH; footprint NetTie:NetTie-2_THT_Pad1.0mm -> NetTie:NetTie-2_Front1.0mm
- NT377: value NT44_L -> NT35_CH; footprint NetTie:NetTie-2_THT_Pad1.0mm -> NetTie:NetTie-2_Front1.0mm
- NT378: value NT45_L -> NT36_CH; footprint NetTie:NetTie-2_THT_Pad1.0mm -> NetTie:NetTie-2_Front1.0mm
- NT379: value NT46_L -> NT37_CH; footprint NetTie:NetTie-2_THT_Pad1.0mm -> NetTie:NetTie-2_Front1.0mm
- NT38: value NT15_D -> NT47_CL; footprint NetTie:NetTie-2_THT_Pad1.0mm -> NetTie:NetTie-2_Front1.0mm
- NT380: value NT47_L -> NT34_CL; footprint NetTie:NetTie-2_THT_Pad1.0mm -> NetTie:NetTie-2_Front1.0mm
- NT381: value NT44_CL -> NT35_CL; footprint NetTie:NetTie-2_THT_Pad1.0mm -> NetTie:NetTie-2_Front1.0mm
- NT382: value NT45_CL -> NT36_CL; footprint Package_TO_SOT_SMD:SOT-23-8 -> NetTie:NetTie-2_Front1.0mm
- NT383: value NT46_CL -> NT37_CL; footprint NetTie:NetTie-2_THT_Pad1.0mm -> NetTie:NetTie-2_Front1.0mm
- NT384: value NT47_CL -> NT3S_RL; footprint NetTie:NetTie-2_THT_Pad1.0mm -> NetTie:NetTie-2_Front1.0mm
- NT385: value NT44_D -> NT3S_CH; footprint NetTie:NetTie-2_THT_Pad1.0mm -> NetTie:NetTie-2_Front1.0mm
- NT386: value NT45_D -> NT3S_NH; footprint NetTie:NetTie-2_THT_Pad1.0mm -> NetTie:NetTie-2_Front1.0mm
- NT387: value NT46_D -> NT3S_RL; footprint NetTie:NetTie-2_THT_Pad1.0mm -> NetTie:NetTie-2_Front1.0mm
- NT388: value NT47_D -> NT3S_CL; footprint NetTie:NetTie-2_THT_Pad1.0mm -> NetTie:NetTie-2_Front1.0mm
- NT389: value NT4S_RL -> NT3S_L1; footprint NetTie:NetTie-2_THT_Pad1.0mm -> NetTie:NetTie-2_Front1.0mm
- NT39: value NT16_D -> NT4S_RL; footprint NetTie:NetTie-2_THT_Pad1.0mm -> NetTie:NetTie-2_Front1.0mm
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Connections:
- K1 pad 10: Net-(D1-Pad2) -> B10_R
- K1 pad 4: Net-(K1-Pad4) -> B10_L
- K1 pad 7: Net-(K1-Pad7) -> B10_H
- K10 pad 10: Net-(D10-Pad2) -> B40_R
- K10 pad 4: Net-(K10-Pad4) -> B40_L
- K10 pad 7: Net-(K10-Pad7) -> B40_H
- K11 pad 10: Net-(D11-Pad2) -> B41_R
- K11 pad 4: Net-(K11-Pad4) -> B41_L
- K11 pad 7: Net-(K11-Pad7) -> B41_H
- K12 pad 10: Net-(D12-Pad2) -> B42_R
- K12 pad 4: Net-(K12-Pad4) -> B42_L
- K12 pad 7: Net-(K12-Pad7) -> B42_H
- K13 pad 10: Net-(D13-Pad2) -> B43_R
- K13 pad 4: Net-(K13-Pad4) -> B43_L
- K13 pad 7: Net-(K13-Pad7) -> B43_H
- K14 pad 10: Net-(D14-Pad2) -> B44_R
- K14 pad 4: Net-(K14-Pad4) -> B44_L
- K14 pad 7: Net-(K14-Pad7) -> B44_H
- K15 pad 10: Net-(D15-Pad2) -> B45_R
- K15 pad 4: Net-(K15-Pad4) -> B45_L
- K15 pad 7: Net-(K15-Pad7) -> B45_H
- K16 pad 10: Net-(D16-Pad2) -> B46_R
- K16 pad 4: Net-(K16-Pad4) -> B46_L
- K16 pad 7: Net-(K16-Pad7) -> B46_H
- K17 pad 10: Net-(D17-Pad2) -> B47_R
- K17 pad 4: Net-(K17-Pad4) -> B47_L
- K17 pad 7: Net-(K17-Pad7) -> B47_H
- K18 pad 10: Net-(D18-Pad2) -> B4S_R
- K2 pad 10: Net-(D2-Pad2) -> unconnected-(K2-Pad10)
- K2 pad 4: Net-(K2-Pad4) -> B11_L
- K2 pad 7: Net-(K2-Pad7) -> B11_H
- K20 pad 10: Net-(D26-Pad2) -> LPR1_R
- K21 pad 2: Net-(D25-Pad2) -> HPR1_R
- K22 pad 10: Net-(D29-Pad2) -> LPR2_R
- K23 pad 1: Net-(K23-Pad1) -> SSR1_R
- K24 pad 10: Net-(D37-Pad2) -> B20_R
- K24 pad 4: Net-(K24-Pad4) -> B20_L
- K24 pad 7: Net-(K24-Pad7) -> B20_H
- K25 pad 10: Net-(D38-Pad2) -> B21_R
- K25 pad 4: Net-(K25-Pad4) -> B21_L
- K25 pad 7: Net-(K25-Pad7) -> B21_H
- K26 pad 10: Net-(D39-Pad2) -> B22_R
- K26 pad 4: Net-(K26-Pad4) -> B22_L
- K26 pad 7: Net-(K26-Pad7) -> B22_H
- K27 pad 10: Net-(D40-Pad2) -> B23_R
- K27 pad 4: Net-(K27-Pad4) -> B23_L
- K27 pad 7: Net-(K27-Pad7) -> B23_H
- K28 pad 10: Net-(D41-Pad2) -> B24_R
- K28 pad 4: Net-(K28-Pad4) -> B24_L
- K28 pad 7: Net-(K28-Pad7) -> B24_H
- K29 pad 10: Net-(D42-Pad2) -> B25_R
- K29 pad 4: Net-(K29-Pad4) -> B25_L
- K29 pad 7: Net-(K29-Pad7) -> B25_H
- K3 pad 10: Net-(D3-Pad2) -> B12_R
- K3 pad 4: Net-(K3-Pad4) -> B12_L
- K3 pad 7: Net-(K3-Pad7) -> B12_H
- K30 pad 10: Net-(D43-Pad2) -> B26_R
- K30 pad 4: Net-(K30-Pad4) -> B26_L
- K30 pad 7: Net-(K30-Pad7) -> B26_H
- K31 pad 10: Net-(D44-Pad2) -> B27_R
- K31 pad 4: Net-(K31-Pad4) -> B27_L
- K31 pad 7: Net-(K31-Pad7) -> B27_H
- K32 pad 10: Net-(D45-Pad2) -> B2S_R
- K33 pad 10: Net-(D46-Pad2) -> B30_R
- K33 pad 4: Net-(K33-Pad4) -> B30_L
- K33 pad 7: Net-(K33-Pad7) -> B30_H
- K34 pad 10: Net-(D47-Pad2) -> unconnected-(K34-Pad10)
- K34 pad 4: Net-(K34-Pad4) -> B31_L
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Routing:
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- added copper zone on In1.Cu, net PWR_5V
Other:
- board size 412 x 195.1 mm -> 479.2 x 749.3 mm
- copper layers 2 -> 4
- board text added: "NT36_LL"

Commit message: Relay bank wired
Parts:
- moved C17 472.6 mm to (781.4, 150.2), turned to -90 degrees
- moved NT353 453.5 mm to (679.0, 256.8), turned to -90 degrees
- moved NT356 452.9 mm to (679.0, 265.1), turned to 90 degrees
- moved NT357 452.8 mm to (679.0, 283.5), turned to 90 degrees
- moved NT358 452.7 mm to (679.0, 275.2), turned to -90 degrees
- moved TP105 446.3 mm to (673.2, 249.2), turned to 0 degrees
- moved NT364 444.0 mm to (672.6, 289.2), turned to 0 degrees
- moved TP106 443.8 mm to (672.6, 268.9), turned to 0 degrees
- moved K30 438.0 mm to (667.8, 254.4), turned to 0 degrees
- moved K32 437.4 mm to (667.8, 293.1), turned to 0 degrees
- moved K31 436.9 mm to (667.8, 274.1), turned to 0 degrees
- moved TP109 433.6 mm to (664.4, 250.6), turned to -90 degrees
- moved NT365 432.4 mm to (663.7, 300.6), turned to -90 degrees
- moved NT360 432.1 mm to (663.7, 255.5), turned to -90 degrees
- moved NT366 431.9 mm to (663.7, 294.9), turned to -90 degrees
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Routing:
- net B35_L: track 0.00 -> 124.8 mm, vias 0 -> 1
- net B35_H: track 0.00 -> 123.5 mm, vias 0 -> 1
- net B3_COM_H: track 0.00 -> 123.4 mm, vias 0 -> 1
- net B3_COM_L: track 0.00 -> 122.0 mm, vias 0 -> 1
- net B34_H: track 0.00 -> 112.2 mm, vias 0 -> 1
- net B37_L: track 0.00 -> 111.5 mm, vias 0 -> 1
- net B34_L: track 0.00 -> 108.7 mm, vias 0 -> 1
- net B37_H: track 0.00 -> 104.6 mm, vias 0 -> 1
- net B36_L: track 0.00 -> 96.9 mm, vias 0 -> 1
- net B33_L: track 0.00 -> 96.0 mm, vias 0 -> 1
- net B33_H: track 0.00 -> 95.7 mm, vias 0 -> 1
- net B36_H: track 0.00 -> 90.1 mm, vias 0 -> 1
- net B42_R: track 85.8 -> 0.00 mm
- net B43_R: track 72.4 -> 0.00 mm
- net B45_R: track 68.5 -> 0.00 mm
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