File: Interconnect.kicad_sch (KiCad schematic)
At the start: 0 parts

Commit message: backup 1 bank done
Other:
- added sheet relay power driver (Relay_driver.kicad_sch)
- note added: "RELAYS DRIVER"
