File: AlertDevice.kicad_sch (KiCad schematic)
At the start: 10 parts, among them Q1 2N2222, Q2 2N2222

Commit message: update
Correction of small error
Parts:
- R2, R3, R69, R71: footprint Resistor_THT:R_Axial_DIN0309_L9.0mm_D3.2mm_P12.70mm_Horizontal -> Resistor_THT:R_Axial_DIN0207_L6.3mm_D2.5mm_P10.16mm_Horizontal
Changed lines of the file:
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@@
     (property "Reference" "R69" (id 0) (at 107.95 55.88 90))
     (property "Value" "120" (id 1) (at 113.03 54.61 90))
-    (property "Footprint" "Resistor_THT:R_Axial_DIN0309_L9.0mm_D3.2mm_P12.70mm_Horizontal" (id 2) (at 109.474 54.356 90)
+    (property "Footprint" "Resistor_THT:R_Axial_DIN0207_L6.3mm_D2.5mm_P10.16mm_Horizontal" (id 2) (at 109.474 54.356 90)
       (effects (font (size 1.27 1.27)) hide)
     )
@@
     (property "Reference" "R71" (id 0) (at 109.22 115.57 0))
     (property "Value" "0" (id 1) (at 118.11 115.57 0))
-    (property "Footprint" "Resistor_THT:R_Axial_DIN0309_L9.0mm_D3.2mm_P12.70mm_Horizontal" (id 2) (at 113.284 114.046 90)
+    (property "Footprint" "Resistor_THT:R_Axial_DIN0207_L6.3mm_D2.5mm_P10.16mm_Horizontal" (id 2) (at 113.284 114.046 90)
       (effects (font (size 1.27 1.27)) hide)
     )
@@
     (property "Reference" "R2" (id 0) (at 57.15 77.47 90))
     (property "Value" "10K" (id 1) (at 57.15 82.55 90))
-    (property "Footprint" "Resistor_THT:R_Axial_DIN0309_L9.0mm_D3.2mm_P12.70mm_Horizontal" (id 2) (at 56.896 81.026 90)
+    (property "Footprint" "Resistor_THT:R_Axial_DIN0207_L6.3mm_D2.5mm_P10.16mm_Horizontal" (id 2) (at 56.896 81.026 90)
       (effects (font (size 1.27 1.27)) hide)
     )
@@
     (property "Reference" "R3" (id 0) (at 69.85 135.89 90))
     (property "Value" "10K" (id 1) (at 69.85 140.97 90))
-    (property "Footprint" "Resistor_THT:R_Axial_DIN0309_L9.0mm_D3.2mm_P12.70mm_Horizontal" (id 2) (at 69.596 139.446 90)
+    (property "Footprint" "Resistor_THT:R_Axial_DIN0207_L6.3mm_D2.5mm_P10.16mm_Horizontal" (id 2) (at 69.596 139.446 90)
       (effects (font (size 1.27 1.27)) hide)
     )
