File: OtherRessource.kicad_sch (KiCad schematic)
At the start: 57 parts, among them K1 TQ2-5, K2 TQ2-5, K3 G5LE-1, K4 CPC1706Y, Q19 2N2222, Q20 2N2222, Q21 2N2222, Q22 2N2222, Q55 2N2222, Q56 2N2222, Q57 2N2222

Commit message: First try to fit electronic on PCB
Parts:
- removed D41, D42, D45, D46: LED, LED_THT:LED_D3.0mm_Clear, symbol Device:LED
- removed R47, R48, R53, R55: 220, Resistor_THT:R_Axial_DIN0309_L9.0mm_D3.2mm_P12.70mm_Horizontal, symbol Device:R_US
- NT399: renamed from NT574; footprint NetTie:NetTie-2_SMD_Pad2.0mm -> NetTie:NetTie-2_THT_Pad1.0mm
- NT401: renamed from NT575; footprint NetTie:NetTie-2_SMD_Pad2.0mm -> NetTie:NetTie-2_THT_Pad1.0mm
- NT403: renamed from NT576; footprint NetTie:NetTie-2_SMD_Pad2.0mm -> NetTie:NetTie-2_THT_Pad1.0mm
- NT405: renamed from NT577; footprint NetTie:NetTie-2_SMD_Pad2.0mm -> NetTie:NetTie-2_THT_Pad1.0mm
- NT409: renamed from NT581; footprint NetTie:NetTie-2_SMD_Pad2.0mm -> NetTie:NetTie-2_THT_Pad1.0mm
- NT412: renamed from NT582; footprint NetTie:NetTie-2_SMD_Pad2.0mm -> NetTie:NetTie-2_THT_Pad1.0mm
- NT420: renamed from NT583; footprint NetTie:NetTie-2_SMD_Pad2.0mm -> NetTie:NetTie-2_THT_Pad1.0mm
- TP73: renamed from TP136; footprint Connector_Pin:Pin_D1.2mm_L11.3mm_W3.0mm_Flat -> Connector_Pin:Pin_D1.0mm_L10.0mm
- TP74: renamed from TP137; footprint Connector_Pin:Pin_D1.2mm_L11.3mm_W3.0mm_Flat -> Connector_Pin:Pin_D1.0mm_L10.0mm
- TP75: renamed from TP138; footprint Connector_Pin:Pin_D1.2mm_L11.3mm_W3.0mm_Flat -> Connector_Pin:Pin_D1.0mm_L10.0mm
- renumbered D43 to D25, D44 to D26, D47 to D29, K1 to K20, K3 to K21, K2 to K22, K4 to K23, NT396 to NT400, NT397 to NT402, NT398 to NT404, NT399 to NT406, NT400 to NT407, NT401 to NT408, NT402 to NT410, NT403 to NT411, NT404 to NT413, NT405 to NT414, NT406 to NT415, NT407 to NT416, NT408 to NT417, NT409 to NT418, NT410 to NT419, NT411 to NT421, Q55 to Q19, Q19 to Q20, Q20 to Q21, Q56 to Q22, Q21 to Q23, Q57 to Q24, Q22 to Q25, R51 to R29, R133 to R31, R49 to R33, R50 to R34, R134 to R35, R52 to R36, R54 to R38, R135 to R40, R56 to R41

Commit message: backup 1 bank done
Parts:
- removed D25, D26, D29: 1N4148, Diode_THT:D_DO-35_SOD27_P7.62mm_Horizontal, symbol Diode:1N4148
- removed NT410: HRL_D, NetTie:NetTie-2_THT_Pad1.0mm, symbol Device:NetTie_2
- removed NT411: LP1_D, NetTie:NetTie-2_THT_Pad1.0mm, symbol Device:NetTie_2
- removed NT419: SSR_D, NetTie:NetTie-2_THT_Pad1.0mm, symbol Device:NetTie_2
- removed NT421: LP2_D, NetTie:NetTie-2_THT_Pad1.0mm, symbol Device:NetTie_2
- removed Q20, Q21, Q23, Q25: 2N2222, Package_TO_SOT_THT:TO-92_Inline, symbol Transistor_BJT:2N3904
- removed R33, R34, R38, R41: 10K, Resistor_THT:R_Axial_DIN0309_L9.0mm_D3.2mm_P12.70mm_Horizontal, symbol Device:R_US
- NT399, NT400, NT401, NT402, NT403, NT404, NT405, NT406, NT407, NT408, NT409, NT412, NT413, NT414, NT415, NT416, NT417, NT418, NT420: footprint NetTie:NetTie-2_THT_Pad1.0mm -> NetTie:NetTie-2_Front1.0mm
- TP73, TP74, TP75: footprint Connector_Pin:Pin_D1.0mm_L10.0mm -> Connector_Pin:Pin_D0.9mm_L10.0mm_W2.4mm_FlatFork
Connections:
- net LPR2_R: now reaches K22.10
- net HPR1_R: now reaches K21.2
- net LPR1_R: now reaches K20.10
- net SSR1_R: now reaches K23.1

Commit message: PCB Completed
PCB completed but final verification not completed
Parts:
- TP73, TP74, TP75: footprint Connector_Pin:Pin_D0.9mm_L10.0mm_W2.4mm_FlatFork -> TestPoint:TestPoint_THTPad_D1.5mm_Drill0.7mm
Changed lines of the file:
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@@
       (effects (font (size 1.27 1.27)) (justify left))
     )
-    (property "Footprint" "Connector_Pin:Pin_D0.9mm_L10.0mm_W2.4mm_FlatFork" (id 2) (at 139.7 41.91 0)
+    (property "Footprint" "TestPoint:TestPoint_THTPad_D1.5mm_Drill0.7mm" (id 2) (at 139.7 41.91 0)
       (effects (font (size 1.27 1.27)) hide)
     )
@@
       (effects (font (size 1.27 1.27)) (justify left))
     )
-    (property "Footprint" "Connector_Pin:Pin_D0.9mm_L10.0mm_W2.4mm_FlatFork" (id 2) (at 154.94 44.45 0)
+    (property "Footprint" "TestPoint:TestPoint_THTPad_D1.5mm_Drill0.7mm" (id 2) (at 154.94 44.45 0)
       (effects (font (size 1.27 1.27)) hide)
     )
@@
       (effects (font (size 1.27 1.27)) (justify left))
     )
-    (property "Footprint" "Connector_Pin:Pin_D0.9mm_L10.0mm_W2.4mm_FlatFork" (id 2) (at 154.94 39.37 0)
+    (property "Footprint" "TestPoint:TestPoint_THTPad_D1.5mm_Drill0.7mm" (id 2) (at 154.94 39.37 0)
       (effects (font (size 1.27 1.27)) hide)
     )

Commit message: update
Correction of small error
Parts:
- K21: value G5LE-1 -> SRD-5VDC-SL-C
- R31, R35, R36, R40: footprint Resistor_THT:R_Axial_DIN0309_L9.0mm_D3.2mm_P12.70mm_Horizontal -> Resistor_THT:R_Axial_DIN0207_L6.3mm_D2.5mm_P10.16mm_Horizontal
Changed lines of the file:
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@@
     (property "Reference" "R31" (id 0) (at 223.52 59.69 90))
     (property "Value" "10K" (id 1) (at 223.52 64.77 90))
-    (property "Footprint" "Resistor_THT:R_Axial_DIN0309_L9.0mm_D3.2mm_P12.70mm_Horizontal" (id 2) (at 223.266 63.246 90)
+    (property "Footprint" "Resistor_THT:R_Axial_DIN0207_L6.3mm_D2.5mm_P10.16mm_Horizontal" (id 2) (at 223.266 63.246 90)
       (effects (font (size 1.27 1.27)) hide)
     )
@@
       (effects (font (size 1.27 1.27)) (justify left))
     )
-    (property "Value" "G5LE-1" (id 1) (at 143.51 30.48 90)
+    (property "Value" "SRD-5VDC-SL-C" (id 1) (at 139.7 54.61 90)
       (effects (font (size 1.27 1.27)) (justify left))
     )
@@
     (property "Reference" "R36" (id 0) (at 146.05 97.79 0))
     (property "Value" "470" (id 1) (at 146.05 100.33 0))
-    (property "Footprint" "Resistor_THT:R_Axial_DIN0309_L9.0mm_D3.2mm_P12.70mm_Horizontal" (id 2) (at 141.224 98.806 90)
+    (property "Footprint" "Resistor_THT:R_Axial_DIN0207_L6.3mm_D2.5mm_P10.16mm_Horizontal" (id 2) (at 141.224 98.806 90)
       (effects (font (size 1.27 1.27)) hide)
     )
@@
     (property "Reference" "R40" (id 0) (at 223.52 127 90))
     (property "Value" "10K" (id 1) (at 223.52 132.08 90))
-    (property "Footprint" "Resistor_THT:R_Axial_DIN0309_L9.0mm_D3.2mm_P12.70mm_Horizontal" (id 2) (at 223.266 130.556 90)
+    (property "Footprint" "Resistor_THT:R_Axial_DIN0207_L6.3mm_D2.5mm_P10.16mm_Horizontal" (id 2) (at 223.266 130.556 90)
       (effects (font (size 1.27 1.27)) hide)
     )
@@
     (property "Reference" "R35" (id 0) (at 223.52 91.44 90))
     (property "Value" "10K" (id 1) (at 223.52 96.52 90))
-    (property "Footprint" "Resistor_THT:R_Axial_DIN0309_L9.0mm_D3.2mm_P12.70mm_Horizontal" (id 2) (at 223.266 94.996 90)
-      (effects (font (size 1.27 1.27)) hide)
-    )
+    (property "Footprint" "Resistor_THT:R_Axial_DIN0207_L6.3mm_D2.5mm_P10.16mm_Horizontal" (id 2) (at 223.266 94.996 90)
+      (effects (font (size 1.27 1.27)) hide)
+    )
