File: communication.kicad_sch (KiCad schematic)
At the start: 68 parts, among them J23 6x2.54mm, J24 6x2.54mm, J25 6x2.54mm, J26 6x2.54mm, J27 6x2.54mm, J28 6x2.54mm, Q23 BSS138, Q24 BSS138, Q25 BSS138, Q26 BSS138, Q27 BSS138, Q28 BSS138, Q29 BSS138, Q30 BSS138, Q31 BSS138, Q32 BSS138, Q33 BSS138, Q34 BSS138

Commit message: First try to fit electronic on PCB
Parts:
- removed J23, J24, J27, J28: 6x2.54mm, Connector_PinHeader_2.54mm:PinHeader_1x06_P2.54mm_Vertical, symbol Connector:Conn_01x06_Male
- removed NT412, NT428: M3_1, NetTie:NetTie-2_THT_Pad1.0mm, symbol Device:NetTie_2
- removed NT413, NT429: M3_H1, NetTie:NetTie-2_THT_Pad1.0mm, symbol Device:NetTie_2
- removed NT416: M3_2, NetTie:NetTie-2_THT_Pad1.0mm, symbol Device:NetTie_2
- removed NT417: M3_H2, NetTie:NetTie-2_THT_Pad1.0mm, symbol Device:NetTie_2
- removed NT420, NT432: M3_3, NetTie:NetTie-2_THT_Pad1.0mm, symbol Device:NetTie_2
- removed NT421, NT433: M3_H3, NetTie:NetTie-2_THT_Pad1.0mm, symbol Device:NetTie_2
- removed NT424: M3_4, NetTie:NetTie-2_THT_Pad1.0mm, symbol Device:NetTie_2
- removed NT425: M3_H4, NetTie:NetTie-2_THT_Pad1.0mm, symbol Device:NetTie_2
- removed Q23, Q25, Q27, Q29, Q31, Q33: BSS138, Package_TO_SOT_SMD:SOT-23, symbol Transistor_FET:BSS138
- removed R57, R66, R69, R70, R73, R74, R75, R76, R77, R78, R79, R80: 10K, Resistor_SMD:R_0603_1608Metric, symbol Device:R_US
- added J11, J12, J15, J16: 6x2.54mm, Connector_PinHeader_2.54mm:PinHeader_1x06_P2.54mm_Vertical, symbol Connector:Conn_01x06_Male
- added NT422: M1_1, NetTie:NetTie-2_THT_Pad1.0mm, symbol Device:NetTie_2
- added NT423: M1_H1, NetTie:NetTie-2_THT_Pad1.0mm, symbol Device:NetTie_2
- added NT426: M1_2, NetTie:NetTie-2_THT_Pad1.0mm, symbol Device:NetTie_2
- added NT427: M1_H2, NetTie:NetTie-2_THT_Pad1.0mm, symbol Device:NetTie_2
- added NT438: M2_1, NetTie:NetTie-2_THT_Pad1.0mm, symbol Device:NetTie_2
- added NT439: M2_H1, NetTie:NetTie-2_THT_Pad1.0mm, symbol Device:NetTie_2
- added NT440: M2_2, NetTie:NetTie-2_THT_Pad1.0mm, symbol Device:NetTie_2
- added NT441: M2_H2, NetTie:NetTie-2_THT_Pad1.0mm, symbol Device:NetTie_2
- added NT442: M2_3, NetTie:NetTie-2_THT_Pad1.0mm, symbol Device:NetTie_2
- added NT443: M2_H3, NetTie:NetTie-2_THT_Pad1.0mm, symbol Device:NetTie_2
- added NT444: M2_4, NetTie:NetTie-2_THT_Pad1.0mm, symbol Device:NetTie_2
- added NT445: M2_H4, NetTie:NetTie-2_THT_Pad1.0mm, symbol Device:NetTie_2
- added Q26, Q28, Q30, Q35, Q36, Q37: BSS138, Package_TO_SOT_SMD:SOT-23W, symbol Transistor_FET:BSS138
- added R42, R43, R46, R47, R50, R51, R54, R55, R59, R60, R63, R64: 10K, Resistor_SMD:R_0603_1608Metric, symbol Device:R_US
- NT430: value M3_2 -> M1_3
- NT431: value M3_H2 -> M1_H3
- NT434: value M3_4 -> M1_4
- NT435: value M3_H4 -> M1_H4
- Q27: renamed from Q24; footprint Package_TO_SOT_SMD:SOT-23 -> Package_TO_SOT_SMD:SOT-23W
- Q29: renamed from Q26; footprint Package_TO_SOT_SMD:SOT-23 -> Package_TO_SOT_SMD:SOT-23W
- Q31: renamed from Q28; footprint Package_TO_SOT_SMD:SOT-23 -> Package_TO_SOT_SMD:SOT-23W
- Q32, Q34: footprint Package_TO_SOT_SMD:SOT-23 -> Package_TO_SOT_SMD:SOT-23W
- Q33: renamed from Q30; footprint Package_TO_SOT_SMD:SOT-23 -> Package_TO_SOT_SMD:SOT-23W
- TP76: renamed from TP24; footprint Connector_PinHeader_2.54mm:PinHeader_1x01_P2.54mm_Vertical -> Connector_Pin:Pin_D1.0mm_L10.0mm
- TP77: renamed from TP26; footprint Connector_PinHeader_2.54mm:PinHeader_1x01_P2.54mm_Vertical -> Connector_Pin:Pin_D1.0mm_L10.0mm
- renumbered J25 to J13, J26 to J14, NT414 to NT424, NT415 to NT425, NT418 to NT428, NT419 to NT429, NT422 to NT432, NT423 to NT433, NT426 to NT436, NT427 to NT437, R59 to R44, R60 to R45, R63 to R48, R64 to R49, R67 to R52, R68 to R53, R71 to R56, R72 to R57
Connections:
- net DIG_PWR_IN: now also R61.2, R65.2, J12.3 (Pin_3), J16.3 (Pin_3), R43.2, R47.2, R51.2, R55.2, R59.2, R63.2; no longer R58.2, R62.2
- net GND: now also J11.4 (Pin_4), J12.4 (Pin_4), J15.4 (Pin_4), J16.4 (Pin_4)
- net M3_HV1: no longer R58.1
- net M3_HV2: no longer NT431.2, Q32.3 (D), R62.1
- net M3_HV4: no longer NT435.2, Q34.3 (D)
- net M3_LV2: no longer NT430.2, Q32.2 (S), R61.1
- net M3_LV3: no longer R65.1
- net M3_LV4: no longer NT434.2, Q34.2 (S)
- net MSR_3V3: now also R58.2, R62.2, J11.3 (Pin_3), J15.3 (Pin_3), Q26.1 (G), Q28.1 (G), Q30.1 (G), Q35.1 (G), Q36.1 (G), Q37.1 (G), R42.2, R46.2, R50.2, R54.2, R60.2, R64.2; no longer R61.2, R65.2
- net SERIAL_CTS: now also NT445.1; no longer NT435.1
- net SERIAL_RTS: now also NT443.1
- net SERIAL_RX: now also NT441.1; no longer NT431.1
- net SERIAL_TX: now also NT439.1
- net SPI0_CLK: now also NT422.1
- net SPI0_CS: now also NT434.1
- net SPI0_RX: now also NT430.1
- net SPI0_TX: now also NT426.1
- net UART1-CTS: now also NT444.1; no longer NT434.1
- net UART1-RTS: now also NT442.1
- net UART1-RX: now also NT440.1; no longer NT430.1
- net UART1-TX: now also NT438.1
- net USPI0_CLK: now also NT423.1
- net USPI0_CS: now also NT435.1
- net USPI0_RX: now also NT431.1
- net USPI0_TX: now also NT427.1
- new net M2_HV1: J12.1 (Pin_1), J16.1 (Pin_1), NT423.2, NT439.2, Q26.3 (D), Q34.3 (D), R43.1, R59.1
- new net M2_HV2: J12.2 (Pin_2), J16.2 (Pin_2), NT427.2, NT441.2, Q28.3 (D), Q35.3 (D), R47.1, R61.1
- new net M2_HV3: J12.5 (Pin_5), J16.5 (Pin_5), NT431.2, NT443.2, Q30.3 (D), Q36.3 (D), R51.1, R63.1
- new net M2_HV4: J12.6 (Pin_6), J16.6 (Pin_6), NT435.2, NT445.2, Q32.3 (D), Q37.3 (D), R55.1, R65.1
- new net M2_LV1: J11.1 (Pin_1), J15.1 (Pin_1), NT422.2, NT438.2, Q26.2 (S), Q34.2 (S), R42.1, R58.1
- new net M2_LV2: J11.2 (Pin_2), J15.2 (Pin_2), NT426.2, NT440.2, Q28.2 (S), Q35.2 (S), R46.1, R60.1
- new net M2_LV3: J11.5 (Pin_5), J15.5 (Pin_5), NT430.2, NT442.2, Q30.2 (S), Q36.2 (S), R50.1, R62.1
- new net M2_LV4: J11.6 (Pin_6), J15.6 (Pin_6), NT434.2, NT444.2, Q32.2 (S), Q37.2 (S), R54.1, R64.1

Commit message: backup 1 bank done
Parts:
- NT422, NT423, NT424, NT425, NT426, NT427, NT428, NT429, NT430, NT431, NT432, NT433, NT434, NT435, NT436, NT437, NT438, NT439, NT440, NT441, NT442, NT443, NT444, NT445: footprint NetTie:NetTie-2_THT_Pad1.0mm -> NetTie:NetTie-2_Front1.0mm
- TP76, TP77: footprint Connector_Pin:Pin_D1.0mm_L10.0mm -> Connector_Pin:Pin_D0.9mm_L10.0mm_W2.4mm_FlatFork
Changed lines of the file:
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@@
       (effects (font (size 1.27 1.27)) (justify left) hide)
     )
-    (property "Footprint" "Connector_Pin:Pin_D1.0mm_L10.0mm" (id 2) (at 246.38 38.1 0)
+    (property "Footprint" "Connector_Pin:Pin_D0.9mm_L10.0mm_W2.4mm_FlatFork" (id 2) (at 246.38 38.1 0)
       (effects (font (size 1.27 1.27)) hide)
     )
@@
     (property "Reference" "NT431" (id 0) (at 105.41 72.39 0))
     (property "Value" "M1_H3" (id 1) (at 105.41 74.93 0))
-    (property "Footprint" "NetTie:NetTie-2_THT_Pad1.0mm" (id 2) (at 105.41 73.66 0)
+    (property "Footprint" "NetTie:NetTie-2_Front1.0mm" (id 2) (at 105.41 73.66 0)
       (effects (font (size 1.27 1.27)) hide)
     )
@@
     (property "Reference" "NT422" (id 0) (at 44.45 35.56 0))
     (property "Value" "M1_1" (id 1) (at 44.45 38.1 0))
-    (property "Footprint" "NetTie:NetTie-2_THT_Pad1.0mm" (id 2) (at 44.45 36.83 0)
+    (property "Footprint" "NetTie:NetTie-2_Front1.0mm" (id 2) (at 44.45 36.83 0)
       (effects (font (size 1.27 1.27)) hide)
     )
@@
     (property "Reference" "NT426" (id 0) (at 44.45 50.8 0))
     (property "Value" "M1_2" (id 1) (at 44.45 53.34 0))
-    (property "Footprint" "NetTie:NetTie-2_THT_Pad1.0mm" (id 2) (at 44.45 52.07 0)
+    (property "Footprint" "NetTie:NetTie-2_Front1.0mm" (id 2) (at 44.45 52.07 0)
       (effects (font (size 1.27 1.27)) hide)
     )
@@
     (property "Reference" "NT434" (id 0) (at 44.45 87.63 0))
     (property "Value" "M1_4" (id 1) (at 44.45 90.17 0))
-    (property "Footprint" "NetTie:NetTie-2_THT_Pad1.0mm" (id 2) (at 44.45 88.9 0)
+    (property "Footprint" "NetTie:NetTie-2_Front1.0mm" (id 2) (at 44.45 88.9 0)
       (effects (font (size 1.27 1.27)) hide)
     )
@@
     (property "Reference" "NT432" (id 0) (at 172.72 73.66 0))
     (property "Value" "M3_3" (id 1) (at 172.72 76.2 0))
-    (property "Footprint" "NetTie:NetTie-2_THT_Pad1.0mm" (id 2) (at 172.72 74.93 0)
+    (property "Footprint" "NetTie:NetTie-2_Front1.0mm" (id 2) (at 172.72 74.93 0)
       (effects (font (size 1.27 1.27)) hide)
     )
@@
     (property "Reference" "NT443" (id 0) (at 105.41 158.75 0))
     (property "Value" "M2_H3" (id 1) (at 105.41 161.29 0))
-    (property "Footprint" "NetTie:NetTie-2_THT_Pad1.0mm" (id 2) (at 105.41 160.02 0)
+    (property "Footprint" "NetTie:NetTie-2_Front1.0mm" (id 2) (at 105.41 160.02 0)
       (effects (font (size 1.27 1.27)) hide)
     )
@@
     (property "Reference" "NT425" (id 0) (at 233.68 36.83 0))
     (property "Value" "M3_H1" (id 1) (at 233.68 39.37 0))
-    (property "Footprint" "NetTie:NetTie-2_THT_Pad1.0mm" (id 2) (at 233.68 38.1 0)
+    (property "Footprint" "NetTie:NetTie-2_Front1.0mm" (id 2) (at 233.68 38.1 0)
       (effects (font (size 1.27 1.27)) hide)
     )
@@
     (property "Reference" "NT445" (id 0) (at 105.41 173.99 0))
     (property "Value" "M2_H4" (id 1) (at 105.41 176.53 0))
-    (property "Footprint" "NetTie:NetTie-2_THT_Pad1.0mm" (id 2) (at 105.41 175.26 0)
+    (property "Footprint" "NetTie:NetTie-2_Front1.0mm" (id 2) (at 105.41 175.26 0)
       (effects (font (size 1.27 1.27)) hide)
     )
@@
     (property "Reference" "NT429" (id 0) (at 233.68 52.07 0))
     (property "Value" "M3_H2" (id 1) (at 233.68 54.61 0))
-    (property "Footprint" "NetTie:NetTie-2_THT_Pad1.0mm" (id 2) (at 233.68 53.34 0)
+    (property "Footprint" "NetTie:NetTie-2_Front1.0mm" (id 2) (at 233.68 53.34 0)
       (effects (font (size 1.27 1.27)) hide)
     )
@@
     (property "Reference" "NT435" (id 0) (at 105.41 87.63 0))
     (property "Value" "M1_H4" (id 1) (at 105.41 90.17 0))
-    (property "Footprint" "NetTie:NetTie-2_THT_Pad1.0mm" (id 2) (at 105.41 88.9 0)
+    (property "Footprint" "NetTie:NetTie-2_Front1.0mm" (id 2) (at 105.41 88.9 0)
       (effects (font (size 1.27 1.27)) hide)
     )
@@
     (property "Reference" "NT442" (id 0) (at 44.45 158.75 0))
     (property "Value" "M2_3" (id 1) (at 44.45 161.29 0))
-    (property "Footprint" "NetTie:NetTie-2_THT_Pad1.0mm" (id 2) (at 44.45 160.02 0)
+    (property "Footprint" "NetTie:NetTie-2_Front1.0mm" (id 2) (at 44.45 160.02 0)
       (effects (font (size 1.27 1.27)) hide)
     )
@@
     (property "Reference" "NT424" (id 0) (at 172.72 36.83 0))
     (property "Value" "M3_1" (id 1) (at 172.72 39.37 0))
-    (property "Footprint" "NetTie:NetTie-2_THT_Pad1.0mm" (id 2) (at 172.72 38.1 0)
+    (property "Footprint" "NetTie:NetTie-2_Front1.0mm" (id 2) (at 172.72 38.1 0)
       (effects (font (size 1.27 1.27)) hide)
     )
@@
     (property "Reference" "NT438" (id 0) (at 44.45 121.92 0))
     (property "Value" "M2_1" (id 1) (at 44.45 124.46 0))
-    (property "Footprint" "NetTie:NetTie-2_THT_Pad1.0mm" (id 2) (at 44.45 123.19 0)
+    (property "Footprint" "NetTie:NetTie-2_Front1.0mm" (id 2) (at 44.45 123.19 0)
       (effects (font (size 1.27 1.27)) hide)
     )
@@
     (property "Reference" "NT441" (id 0) (at 105.41 137.16 0))
     (property "Value" "M2_H2" (id 1) (at 105.41 139.7 0))
-    (property "Footprint" "NetTie:NetTie-2_THT_Pad1.0mm" (id 2) (at 105.41 138.43 0)
+    (property "Footprint" "NetTie:NetTie-2_Front1.0mm" (id 2) (at 105.41 138.43 0)
       (effects (font (size 1.27 1.27)) hide)
     )
@@
     (property "Reference" "NT440" (id 0) (at 44.45 137.16 0))
     (property "Value" "M2_2" (id 1) (at 44.45 139.7 0))
-    (property "Footprint" "NetTie:NetTie-2_THT_Pad1.0mm" (id 2) (at 44.45 138.43 0)
+    (property "Footprint" "NetTie:NetTie-2_Front1.0mm" (id 2) (at 44.45 138.43 0)
       (effects (font (size 1.27 1.27)) hide)
     )
@@
     (property "Reference" "NT423" (id 0) (at 105.41 35.56 0))
     (property "Value" "M1_H1" (id 1) (at 105.41 38.1 0))
-    (property "Footprint" "NetTie:NetTie-2_THT_Pad1.0mm" (id 2) (at 105.41 36.83 0)
+    (property "Footprint" "NetTie:NetTie-2_Front1.0mm" (id 2) (at 105.41 36.83 0)
       (effects (font (size 1.27 1.27)) hide)
     )
@@
     (property "Reference" "NT430" (id 0) (at 44.45 72.39 0))
     (property "Value" "M1_3" (id 1) (at 44.45 74.93 0))
-    (property "Footprint" "NetTie:NetTie-2_THT_Pad1.0mm" (id 2) (at 44.45 73.66 0)
+    (property "Footprint" "NetTie:NetTie-2_Front1.0mm" (id 2) (at 44.45 73.66 0)
       (effects (font (size 1.27 1.27)) hide)
     )
@@
     (property "Reference" "NT428" (id 0) (at 172.72 52.07 0))
     (property "Value" "M3_2" (id 1) (at 172.72 54.61 0))
-    (property "Footprint" "NetTie:NetTie-2_THT_Pad1.0mm" (id 2) (at 172.72 53.34 0)
+    (property "Footprint" "NetTie:NetTie-2_Front1.0mm" (id 2) (at 172.72 53.34 0)
       (effects (font (size 1.27 1.27)) hide)
     )
@@
     (property "Reference" "NT433" (id 0) (at 233.68 73.66 0))
     (property "Value" "M3_H3" (id 1) (at 233.68 76.2 0))
-    (property "Footprint" "NetTie:NetTie-2_THT_Pad1.0mm" (id 2) (at 233.68 74.93 0)
+    (property "Footprint" "NetTie:NetTie-2_Front1.0mm" (id 2) (at 233.68 74.93 0)
       (effects (font (size 1.27 1.27)) hide)
     )
@@
       (effects (font (size 1.27 1.27)) (justify left) hide)
     )
-    (property "Footprint" "Connector_Pin:Pin_D1.0mm_L10.0mm" (id 2) (at 166.37 38.1 0)
+    (property "Footprint" "Connector_Pin:Pin_D0.9mm_L10.0mm_W2.4mm_FlatFork" (id 2) (at 166.37 38.1 0)
       (effects (font (size 1.27 1.27)) hide)
     )
@@
     (property "Reference" "NT437" (id 0) (at 233.68 88.9 0))
     (property "Value" "M3_H4" (id 1) (at 233.68 91.44 0))
-    (property "Footprint" "NetTie:NetTie-2_THT_Pad1.0mm" (id 2) (at 233.68 90.17 0)
+    (property "Footprint" "NetTie:NetTie-2_Front1.0mm" (id 2) (at 233.68 90.17 0)
       (effects (font (size 1.27 1.27)) hide)
     )
@@
     (property "Reference" "NT436" (id 0) (at 172.72 88.9 0))
     (property "Value" "M3_4" (id 1) (at 172.72 91.44 0))
-    (property "Footprint" "NetTie:NetTie-2_THT_Pad1.0mm" (id 2) (at 172.72 90.17 0)
+    (property "Footprint" "NetTie:NetTie-2_Front1.0mm" (id 2) (at 172.72 90.17 0)
       (effects (font (size 1.27 1.27)) hide)
     )
@@
     (property "Reference" "NT439" (id 0) (at 105.41 121.92 0))
     (property "Value" "M2_H1" (id 1) (at 105.41 124.46 0))
-    (property "Footprint" "NetTie:NetTie-2_THT_Pad1.0mm" (id 2) (at 105.41 123.19 0)
+    (property "Footprint" "NetTie:NetTie-2_Front1.0mm" (id 2) (at 105.41 123.19 0)
       (effects (font (size 1.27 1.27)) hide)
     )
@@
     (property "Reference" "NT444" (id 0) (at 44.45 173.99 0))
     (property "Value" "M2_4" (id 1) (at 44.45 176.53 0))
-    (property "Footprint" "NetTie:NetTie-2_THT_Pad1.0mm" (id 2) (at 44.45 175.26 0)
+    (property "Footprint" "NetTie:NetTie-2_Front1.0mm" (id 2) (at 44.45 175.26 0)
       (effects (font (size 1.27 1.27)) hide)
     )
@@
     (property "Reference" "NT427" (id 0) (at 105.41 50.8 0))
     (property "Value" "M1_H2" (id 1) (at 105.41 53.34 0))
-    (property "Footprint" "NetTie:NetTie-2_THT_Pad1.0mm" (id 2) (at 105.41 52.07 0)
-      (effects (font (size 1.27 1.27)) hide)
-    )
+    (property "Footprint" "NetTie:NetTie-2_Front1.0mm" (id 2) (at 105.41 52.07 0)
+      (effects (font (size 1.27 1.27)) hide)
+    )
