File: InterconnectIO_bd/AlertDevice.kicad_sch (KiCad schematic)
At the start: 10 parts, among them Q1 2N2222, Q2 2N2222

Commit message: Change TO-92 package to 2.54mm package
Transistor and voltage reference using TO-92 Package will have the possibility to be mounted on in-line 3 pins socket of 2.54mm.
Parts:
- Q1, Q2: footprint Package_TO_SOT_THT:TO-92L_HandSolder -> Package_TO_SOT_THT:TO-92_Inline_Wide
Changed lines of the file:
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@@
       (effects (font (size 1.27 1.27)))
     )
-    (property "Footprint" "Package_TO_SOT_THT:TO-92L_HandSolder" (at 85.09 140.335 0)
+    (property "Footprint" "Package_TO_SOT_THT:TO-92_Inline_Wide" (at 85.09 140.335 0)
       (effects (font (size 1.27 1.27) italic) (justify left) hide)
     )
@@
       (effects (font (size 1.27 1.27)))
     )
-    (property "Footprint" "Package_TO_SOT_THT:TO-92L_HandSolder" (at 72.39 81.915 0)
+    (property "Footprint" "Package_TO_SOT_THT:TO-92_Inline_Wide" (at 72.39 81.915 0)
       (effects (font (size 1.27 1.27) italic) (justify left) hide)
     )
