File: InterconnectIO_bd/MainInput.kicad_sch (KiCad schematic)
At the start: 33 parts, among them J27 PJ-082BH, J28 DB9_Female_RA, J29 Conn_01x04_Female, J34 Conn_01x04_Female, J35 Conn_01x03_Male, K21 SRD-5VDC-SL-C, Q5 2N2222, U9 MAX3232

Commit message: Change TO-92 package to 2.54mm package
Transistor and voltage reference using TO-92 Package will have the possibility to be mounted on in-line 3 pins socket of 2.54mm.
Parts:
- Q5: footprint Package_TO_SOT_THT:TO-92L_HandSolder -> Package_TO_SOT_THT:TO-92_Inline_Wide
Changed lines of the file:
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@@
       (effects (font (size 1.27 1.27)))
     )
-    (property "Footprint" "Package_TO_SOT_THT:TO-92L_HandSolder" (at 177.8 61.595 0)
+    (property "Footprint" "Package_TO_SOT_THT:TO-92_Inline_Wide" (at 177.8 61.595 0)
       (effects (font (size 1.27 1.27) italic) (justify left) hide)
     )
