File: InterconnectIO_bd/OtherRessource.kicad_sch (KiCad schematic)
At the start: 34 parts, among them K20 TQ2-5, K21 SRD-5VDC-SL-C, K22 TQ2-5, K23 CPC1706Y, Q19 2N2222, Q22 2N2222, Q24 2N2222

Commit message: Change TO-92 package to 2.54mm package
Transistor and voltage reference using TO-92 Package will have the possibility to be mounted on in-line 3 pins socket of 2.54mm.
Parts:
- Q19, Q22, Q24: footprint Package_TO_SOT_THT:TO-92L_HandSolder -> Package_TO_SOT_THT:TO-92_Inline_Wide
Changed lines of the file:
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@@
       (effects (font (size 1.27 1.27)))
     )
-    (property "Footprint" "Package_TO_SOT_THT:TO-92L_HandSolder" (at 238.76 131.445 0)
+    (property "Footprint" "Package_TO_SOT_THT:TO-92_Inline_Wide" (at 238.76 131.445 0)
       (effects (font (size 1.27 1.27) italic) (justify left) hide)
     )
@@
       (effects (font (size 1.27 1.27)))
     )
-    (property "Footprint" "Package_TO_SOT_THT:TO-92L_HandSolder" (at 238.76 64.135 0)
+    (property "Footprint" "Package_TO_SOT_THT:TO-92_Inline_Wide" (at 238.76 64.135 0)
       (effects (font (size 1.27 1.27) italic) (justify left) hide)
     )
@@
       (effects (font (size 1.27 1.27)))
     )
-    (property "Footprint" "Package_TO_SOT_THT:TO-92L_HandSolder" (at 238.76 95.885 0)
+    (property "Footprint" "Package_TO_SOT_THT:TO-92_Inline_Wide" (at 238.76 95.885 0)
       (effects (font (size 1.27 1.27) italic) (justify left) hide)
     )
