File: InterconnectIO_bd/Pmaster.kicad_sch (KiCad schematic)
At the start: 161 parts, among them U1 Pico, U2 Pico, U3 Pico, U4 Pico, U5 LM4040LP-3

Commit message: Change TO-92 package to 2.54mm package
Transistor and voltage reference using TO-92 Package will have the possibility to be mounted on in-line 3 pins socket of 2.54mm.
Parts:
- U5: footprint Package_TO_SOT_THT:TO-92_Inline -> Package_TO_SOT_THT:TO-92_Inline_Wide
Changed lines of the file:
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@@
       (effects (font (size 1.27 1.27)) (justify right))
     )
-    (property "Footprint" "Package_TO_SOT_THT:TO-92_Inline" (at 144.78 72.39 0)
+    (property "Footprint" "Package_TO_SOT_THT:TO-92_Inline_Wide" (at 144.78 72.39 0)
       (effects (font (size 1.27 1.27) italic) hide)
     )
