File: InterconnectIO_bd/protection.kicad_sch (KiCad schematic)
At the start: 34 parts, among them J10 10x2.54mm, J5 10x2.54mm, J6 10x2.54mm, J7 10x2.54mm, J8 10x2.54mm, J9 10x2.54mm, K19 TQ2-5, Q3 2N2222, U6 TXS0108EPW, U7 TXS0108EPW, U8 TXS0108EPW

Commit message: Change TO-92 package to 2.54mm package
Transistor and voltage reference using TO-92 Package will have the possibility to be mounted on in-line 3 pins socket of 2.54mm.
Parts:
- Q3: footprint Package_TO_SOT_THT:TO-92L_HandSolder -> Package_TO_SOT_THT:TO-92_Inline_Wide
Changed lines of the file:
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@@
       (effects (font (size 1.27 1.27)))
     )
-    (property "Footprint" "Package_TO_SOT_THT:TO-92L_HandSolder" (at 55.88 188.595 0)
+    (property "Footprint" "Package_TO_SOT_THT:TO-92_Inline_Wide" (at 55.88 188.595 0)
       (effects (font (size 1.27 1.27) italic) (justify left) hide)
     )
